Commit message: got movo working with inverse dynamics in drake w/o any hands

File: movo_common/movo_description/urdf/manipulation/kinova_grippers/kg2_gripper.urdf.xacro (robot description, xacro)
@@ -197,4 +197,16 @@
             </collision>
             <inertial>
+                <!-- russt: set these using drake's mesh to sdf -->
+                <pose>0.0148543 -0.00150728 -1.56703e-09 0 0 0</pose>
+                <mass>0.012779909194886162</mass>
+                <inertia>
+                  <ixx>1.05756e-06</ixx>
+                  <ixy>-9.59984e-07</ixy>
+                  <ixz>2.26386e-13</ixz>
+                  <iyy>3.44081e-06</iyy>
+                  <iyz>-1.09241e-14</iyz>
+                  <izz>3.8057e-06</izz>
+                </inertia>
+                <!-- these original values aren't physically valid
                 <mass value="0.012690" />
                 <origin xyz="-0.011926 -0.009701 0.0" />
@@ -202,4 +214,5 @@
                          iyx = "0.000001" iyy = "0.000001" iyz = "0.000000"
                          izx = "0.000000" izy = "0.000000" izz = "0.000002" />
+                -->
             </inertial>
         </link>

File: movo_common/movo_description/urdf/manipulation/kinova_grippers/kg3_gripper.transmission.xacro (robot description, xacro)
@@ -12,4 +12,26 @@
             </actuator>
         </transmission>
+        <!-- russt: add extra transmissions to avoid mimic joints -->
+        <transmission name="${prefix}gripper_finger2_trans">
+            <type>transmission_interface/SimpleTransmission</type>
+            <joint name="${prefix}gripper_finger2_joint">
+                <hardwareInterface>EffortJointInterface</hardwareInterface>
+            </joint>
+            <actuator name="${prefix}gripper_finger2_motor">
+                <mechanicalReduction>1</mechanicalReduction>
+                <hardwareInterface>EffortJointInterface</hardwareInterface>
+            </actuator>
+        </transmission>
+        <transmission name="${prefix}gripper_finger3_trans">
+            <type>transmission_interface/SimpleTransmission</type>
+            <joint name="${prefix}gripper_finger3_joint">
+                <hardwareInterface>EffortJointInterface</hardwareInterface>
+            </joint>
+            <actuator name="${prefix}gripper_finger3_motor">
+                <mechanicalReduction>1</mechanicalReduction>
+                <hardwareInterface>EffortJointInterface</hardwareInterface>
+            </actuator>
+        </transmission>
+        <!-- end of extra transmissions -->
         <gazebo>
                 <!-- loading plugin: mimic joints works in gazebo now -->

File: movo_common/movo_description/urdf/manipulation/kinova_grippers/kg3_gripper.urdf.xacro (robot description, xacro)
@@ -91,5 +91,5 @@
             <origin rpy="${M_PI/2} 0 1.7555" xyz="0.022289 -0.027253 -0.11471"/>
             <limit lower="0.0" upper="0.986111027" velocity="1.0" effort="3.0" damping="0.005" friction="0.005"/>
-            <mimic joint="${prefix}gripper_finger1_joint"/>
+            <!-- <mimic joint="${prefix}gripper_finger1_joint"/> -->
         </joint>
         <link name="${prefix}gripper_finger2_knuckle_link">
@@ -140,5 +140,5 @@
             <origin rpy="${M_PI/2} 0 1.3861" xyz="-0.022284 -0.027223 -0.11473"/>
             <limit lower="0.0" upper="0.986111027" velocity="1.0" effort="3.0" damping="0.005" friction="0.005"/>
-            <mimic joint="${prefix}gripper_finger1_joint"/>
+            <!-- <mimic joint="${prefix}gripper_finger1_joint"/> -->
         </joint>
         <link name="${prefix}gripper_finger3_knuckle_link">

File: movo_common/movo_description/urdf/movo.urdf.xacro (robot description, xacro)
@@ -71,5 +71,7 @@
     <xacro:if value="$(optenv MOVO_HAS_KINOVA_ARM false)">
     	<xacro:if value="$(optenv MOVO_HAS_KINOVA_ARM_7DOF false)">
-    		<xacro:include filename="$(find movo_description)/urdf/manipulation/jaco/jaco_7dof.urdf.xacro" />
+        <xacro:include filename="$(find movo_description)/urdf/manipulation/jaco/j2s7s300_arm_sphere_collision.urdf.xacro" />
+        <!-- russt: use Drake's jaco 7 dof model
+    		<xacro:include filename="$(find movo_description)/urdf/manipulation/jaco/jaco_7dof.urdf.xacro" /> -->
             <xacro:jaco_robot_7dof prefix="right_" parent="linear_actuator_link">
             <origin xyz="0.0261046 -0.13335 0.2799937" rpy="${-M_PI/2} 0 ${-M_PI/2}"/>

File: movo_common/movo_description/urdf/movo_components/movo_base.urdf.xacro (robot description, xacro)
@@ -131,4 +131,5 @@
                          izx="0.053722" izy="-0.000058" izz="0.098853" />
 			</inertial>
+        <!-- russt: removed this because it was causing self collisions
             <collision>
 				<geometry>
@@ -136,4 +137,5 @@
 				</geometry>
 			</collision>
+      -->
 			<visual>
 				<origin xyz="0 0 0" rpy="0 0 0" />
@@ -160,4 +162,5 @@
 			    </geometry>
 		    </visual>
+        <!-- russt: removed this because it was causing self-collisions
 		    <collision>
 			    <geometry>
@@ -165,4 +168,5 @@
 			    </geometry>
 		    </collision>
+        -->
 	        <inertial>
                 <mass value="12.926242" />

File: movo_common/movo_description/urdf/movo_components/movo_body.urdf.xacro (robot description, xacro)
@@ -72,5 +72,8 @@
 			</visual>
 		</link>
+        <!-- russt: make this fixed for now; it was causing problems with the inverse dynamics controllers.
         <joint name="mid_body_joint" type="prismatic">
+        -->
+        <joint name="mid_body_joint" type="fixed">
             <parent link="base_chassis_link" />
             <child link = "mid_body_link" />
@@ -79,6 +82,16 @@
             <limit lower="0.0" upper="0.2545608" effort="1000" velocity="0.20"/>
             <dynamics damping="0.0" friction="0.0"/>
-            <mimic joint="linear_joint" multiplier="0.5" offset="0.0" />
+            <!-- <mimic joint="linear_joint" multiplier="0.5" offset="0.0" /> -->
         </joint>
+        <!-- russt: add transmission to avoid mimic joint
+        <transmission name="mid_body_trans">
+            <type>transmission_interface/SimpleTransmission</type>
+            <joint name="mid_body_joint">
+                <hardwareInterface>PositionJointInterface</hardwareInterface>
+            </joint>
+            <actuator name="mid_body_motor">
+                <mechanicalReduction>1</mechanicalReduction>
+            </actuator>
+        </transmission>  -->
         <link name="mid_body_link">
 			<inertial>
