Commit message: add WELD_FINGERS xacro logic

File: movo_common/movo_description/urdf/manipulation/robotiq/robotiq_85_gripper.transmission.xacro (robot description, xacro)
@@ -2,60 +2,16 @@
 <robot xmlns:xacro="http://ros.org/wiki/xacro">
   <xacro:macro name="robotiq_85_gripper_transmission" params="prefix">
-        <!-- russt: i've fixed this joint
-        <transmission name="${prefix}gripper_finger1_trans">
-            <type>transmission_interface/SimpleTransmission</type>
-            <joint name="${prefix}gripper_finger1_joint">
-                <hardwareInterface>PositionJointInterface</hardwareInterface>
-            </joint>
-            <actuator name="${prefix}gripper_finger1_motor">
-                <mechanicalReduction>1</mechanicalReduction>
-                <hardwareInterface>PositionJointInterface</hardwareInterface>
-            </actuator>
-        </transmission>
-        -->
-        <!-- russt: add extra transmissions to overcome missing mimic joints -->
-        <!--
-        <transmission name="${prefix}gripper_finger1_inner_knuckle_trans">
-            <type>transmission_interface/SimpleTransmission</type>
-            <joint name="${prefix}gripper_finger1_inner_knuckle_joint">
-                <hardwareInterface>PositionJointInterface</hardwareInterface>
-            </joint>
-            <actuator name="${prefix}gripper_finger1_inner_knuckle_motor">
-                <mechanicalReduction>1</mechanicalReduction>
-                <hardwareInterface>PositionJointInterface</hardwareInterface>
-            </actuator>
-        </transmission>
-        <transmission name="${prefix}gripper_finger2_inner_knuckle_trans">
-            <type>transmission_interface/SimpleTransmission</type>
-            <joint name="${prefix}gripper_finger2_inner_knuckle_joint">
-                <hardwareInterface>PositionJointInterface</hardwareInterface>
-            </joint>
-            <actuator name="${prefix}gripper_finger2_inner_knuckle_motor">
-                <mechanicalReduction>1</mechanicalReduction>
-                <hardwareInterface>PositionJointInterface</hardwareInterface>
-            </actuator>
-        </transmission>
-        <transmission name="${prefix}gripper_finger1_finger_tip_trans">
-            <type>transmission_interface/SimpleTransmission</type>
-            <joint name="${prefix}gripper_finger1_finger_tip_joint">
-                <hardwareInterface>PositionJointInterface</hardwareInterface>
-            </joint>
-            <actuator name="${prefix}gripper_finger1_finger_tip_motor">
-                <mechanicalReduction>1</mechanicalReduction>
-                <hardwareInterface>PositionJointInterface</hardwareInterface>
-            </actuator>
-        </transmission>
-        <transmission name="${prefix}gripper_finger2_finger_tip_trans">
-            <type>transmission_interface/SimpleTransmission</type>
-            <joint name="${prefix}gripper_finger2_finger_tip_joint">
-                <hardwareInterface>PositionJointInterface</hardwareInterface>
-            </joint>
-            <actuator name="${prefix}gripper_finger2_finger_tip_motor">
-                <mechanicalReduction>1</mechanicalReduction>
-                <hardwareInterface>PositionJointInterface</hardwareInterface>
-            </actuator>
-        </transmission>
-        -->
-        <!-- russt: end new transmissions -->
+        <xacro:unless value="$(optenv WELD_FINGERS false)">
+          <transmission name="${prefix}gripper_finger1_trans">
+              <type>transmission_interface/SimpleTransmission</type>
+              <joint name="${prefix}gripper_finger1_joint">
+                  <hardwareInterface>PositionJointInterface</hardwareInterface>
+              </joint>
+              <actuator name="${prefix}gripper_finger1_motor">
+                  <mechanicalReduction>1</mechanicalReduction>
+                  <hardwareInterface>PositionJointInterface</hardwareInterface>
+              </actuator>
+          </transmission>
+        </xacro:unless>
         <gazebo>
                 <!-- loading plugin: mimic joints works in gazebo now -->

File: movo_common/movo_description/urdf/manipulation/robotiq/robotiq_85_gripper.urdf.xacro (robot description, xacro)
@@ -3,4 +3,10 @@
     <xacro:include filename="$(find movo_description)/urdf/manipulation/robotiq/robotiq_85_gripper.transmission.xacro" />
     <xacro:property name="M_PI" value="3.14159"/>
+    <xacro:if value="$(optenv WELD_FINGERS false)">
+      <xacro:property name="revolute_or_fixed" value="fixed"/>
+    </xacro:if>
+    <xacro:unless value="$(optenv WELD_FINGERS false)">
+      <xacro:property name="revolute_or_fixed" value="revolute"/>
+    </xacro:unless>
     <xacro:macro name="robotiq_85_gripper" params="prefix parent *origin">
         <joint name="${prefix}kinova_robotiq_coupler_joint" type="fixed">
@@ -66,7 +72,5 @@
             <kd>1.0</kd>
         </gazebo>
-        <!-- russt: fix this to overcome mimic
-        <joint name="${prefix}gripper_finger1_joint" type="revolute"> -->
-        <joint name="${prefix}gripper_finger1_joint" type="fixed">
+        <joint name="${prefix}gripper_finger1_joint" type="${revolute_or_fixed}">
             <parent link="${prefix}gripper_base_link"/>
             <child link="${prefix}gripper_finger1_knuckle_link"/>
@@ -75,7 +79,5 @@
             <limit lower="0.0" upper="0.804" velocity="2.0" effort="1000"/>
         </joint>
-        <!-- russt: fix this to overcome mimic
-        <joint name="${prefix}gripper_finger2_joint" type="revolute"> -->
-        <joint name="${prefix}gripper_finger2_joint" type="fixed">
+        <joint name="${prefix}gripper_finger2_joint" type="${revolute_or_fixed}">
             <parent link="${prefix}gripper_base_link"/>
             <child link="${prefix}gripper_finger2_knuckle_link"/>
@@ -83,5 +85,7 @@
             <origin rpy="0.0 0.0 0.0" xyz="0.05490451627 -0.03060114443 0.0"/>
             <limit lower="-3.14" upper="3.14" velocity="100.0" effort="1000"/>
-            <!-- russt: remove this until inverse dynamics supports it <mimic joint="${prefix}gripper_finger1_joint"/> -->
+            <xacro:unless value="$(optenv WELD_FINGERS false)">
+              <mimic joint="${prefix}gripper_finger1_joint"/>
+            </xacro:unless>
         </joint>
         <link name="${prefix}gripper_finger1_knuckle_link">
@@ -199,7 +203,5 @@
             <kd>1.0</kd>
         </gazebo>
-        <!-- russt: fix this for now
-        <joint name="${prefix}gripper_finger1_inner_knuckle_joint" type="continuous"> -->
-        <joint name="${prefix}gripper_finger1_inner_knuckle_joint" type="fixed">
+        <joint name="${prefix}gripper_finger1_inner_knuckle_joint" type="${revolute_or_fixed}">
             <parent link="${prefix}gripper_base_link"/>
             <child link="${prefix}gripper_finger1_inner_knuckle_link"/>
@@ -207,11 +209,9 @@
             <origin xyz="0.06142 0.0127 0" rpy="${M_PI} 0.0 0.0" />
             <limit lower="-3.14" upper="3.14" velocity="100.0" effort="0.1"/>
-            <!-- russt: remove this for now
-            <mimic joint="${prefix}gripper_finger1_joint" offset="0"/>
-            -->
-        </joint>
-        <!-- russt: fix this for now
-        <joint name="${prefix}gripper_finger2_inner_knuckle_joint" type="continuous"> -->
-        <joint name="${prefix}gripper_finger2_inner_knuckle_joint" type="fixed">
+            <xacro:unless value="$(optenv WELD_FINGERS false)">
+              <mimic joint="${prefix}gripper_finger1_joint" offset="0"/>
+            </xacro:unless>
+        </joint>
+        <joint name="${prefix}gripper_finger2_inner_knuckle_joint" type="${revolute_or_fixed}">
             <parent link="${prefix}gripper_base_link"/>
             <child link="${prefix}gripper_finger2_inner_knuckle_link"/>
@@ -219,7 +219,7 @@
             <origin xyz="0.06142 -0.0127 0" rpy="0 0 0"/>
             <limit lower="-3.14" upper="3.14" velocity="100.0" effort="0.1"/>
-            <!-- russt: remove this for now
-            <mimic joint="${prefix}gripper_finger1_joint" offset="0"/>
-            -->
+            <xacro:unless value="$(optenv WELD_FINGERS false)">
+              <mimic joint="${prefix}gripper_finger1_joint" offset="0"/>
+            </xacro:unless>
         </joint>
         <link name="${prefix}gripper_finger1_inner_knuckle_link">
@@ -275,7 +275,5 @@
             <kd>1.0</kd>
         </gazebo>
-        <!-- russt: fix this for now
-        <joint name="${prefix}gripper_finger1_finger_tip_joint" type="continuous">-->
-        <joint name="${prefix}gripper_finger1_finger_tip_joint" type="fixed">
+        <joint name="${prefix}gripper_finger1_finger_tip_joint" type="${revolute_or_fixed}">
             <parent link="${prefix}gripper_finger1_inner_knuckle_link"/>
             <child link="${prefix}gripper_finger1_finger_tip_link"/>
@@ -283,11 +281,9 @@
             <origin xyz="0.04303959807 -0.03759940821 0.0" rpy="0.0 0.0 0.0"/>
             <limit lower="-3.14" upper="3.14" velocity="100.0" effort="0.1"/>
-            <!-- russt: remove this for now
-            <mimic joint="${prefix}gripper_finger1_joint" multiplier="-1"/>
-            -->
-        </joint>
-        <!-- russt: fix this for now
-        <joint name="${prefix}gripper_finger2_finger_tip_joint" type="continuous"> -->
-        <joint name="${prefix}gripper_finger2_finger_tip_joint" type="fixed">
+            <xacro:unless value="$(optenv WELD_FINGERS false)">
+              <mimic joint="${prefix}gripper_finger1_joint" multiplier="-1"/>
+            </xacro:unless>
+        </joint>
+        <joint name="${prefix}gripper_finger2_finger_tip_joint" type="${revolute_or_fixed}">
             <parent link="${prefix}gripper_finger2_inner_knuckle_link"/>
             <child link="${prefix}gripper_finger2_finger_tip_link"/>
@@ -295,7 +291,7 @@
             <origin rpy="0.0 0.0 0.0" xyz="0.04303959807 -0.03759940821  0.0"/>
             <limit lower="-3.14" upper="3.14" velocity="100.0" effort="0.1"/>
-            <!-- russt: remove this for now
-            <mimic joint="${prefix}gripper_finger1_joint" multiplier="-1"/>
-            -->
+            <xacro:unless value="$(optenv WELD_FINGERS false)">
+              <mimic joint="${prefix}gripper_finger1_joint" multiplier="-1"/>
+            </xacro:unless>
         </joint>
         <link name="${prefix}gripper_finger1_finger_tip_link">

File: movo_common/movo_description/urdf/movo_components/movo_base.urdf.xacro (robot description, xacro)
@@ -88,5 +88,5 @@
         </gazebo>
         <joint name="base_chassis_joint" type="fixed">
-            <origin xyz="0 0 ${wheel_radius}" rpy="0 0 0" />
+            <origin xyz="0 0 ${wheel_radius + 0.01}" rpy="0 0 0" />
             <parent link="base_link" />
             <child link="base_chassis_link" />
