Commit message: replace dae with obj

File: movo_common/movo_description/urdf/manipulation/robotiq/robotiq_85_gripper.transmission.xacro (robot description, xacro)
@@ -2,4 +2,27 @@
 <robot xmlns:xacro="http://ros.org/wiki/xacro">
   <xacro:macro name="robotiq_85_gripper_transmission" params="prefix">
+        <xacro:if value="$(optenv REPLACE_MIMIC false)">
+          <transmission name="${prefix}gripper_finger1_trans">
+              <type>transmission_interface/SimpleTransmission</type>
+              <joint name="${prefix}gripper_finger1_inner_knuckle_joint">
+                  <hardwareInterface>PositionJointInterface</hardwareInterface>
+              </joint>
+              <actuator name="${prefix}gripper_finger1_motor">
+                  <mechanicalReduction>1</mechanicalReduction>
+                  <hardwareInterface>PositionJointInterface</hardwareInterface>
+              </actuator>
+          </transmission>
+          <transmission name="${prefix}gripper_finger2_trans">
+              <type>transmission_interface/SimpleTransmission</type>
+              <joint name="${prefix}gripper_finger2_inner_knuckle_joint">
+                  <hardwareInterface>PositionJointInterface</hardwareInterface>
+              </joint>
+              <actuator name="${prefix}gripper_finger2_motor">
+                  <mechanicalReduction>1</mechanicalReduction>
+                  <hardwareInterface>PositionJointInterface</hardwareInterface>
+              </actuator>
+          </transmission>
+        </xacro:if>
+        <xacro:unless value="$(optenv REPLACE_MIMIC false)">
         <xacro:unless value="$(optenv WELD_FINGERS false)">
           <transmission name="${prefix}gripper_finger1_trans">
@@ -13,4 +36,5 @@
               </actuator>
           </transmission>
+        </xacro:unless>
         </xacro:unless>
         <gazebo>

File: movo_common/movo_description/urdf/manipulation/robotiq/robotiq_85_gripper.urdf.xacro (robot description, xacro)
@@ -3,9 +3,15 @@
     <xacro:include filename="$(find movo_description)/urdf/manipulation/robotiq/robotiq_85_gripper.transmission.xacro" />
     <xacro:property name="M_PI" value="3.14159"/>
+    <xacro:if value="$(optenv REPLACE_MIMIC false)">
+      <xacro:property name="revolute_or_fixed_1" value="fixed"/>
+    </xacro:if>
+    <xacro:unless value="$(optenv REPLACE_MIMIC false)">
+      <xacro:property name="revolute_or_fixed_1" value="revolute"/>
+    </xacro:unless>
     <xacro:if value="$(optenv WELD_FINGERS false)">
-      <xacro:property name="revolute_or_fixed" value="fixed"/>
+      <xacro:property name="revolute_or_fixed" value="${revolute_or_fixed_1}"/>
     </xacro:if>
     <xacro:unless value="$(optenv WELD_FINGERS false)">
-      <xacro:property name="revolute_or_fixed" value="revolute"/>
+      <xacro:property name="revolute_or_fixed" value="${revolute_or_fixed_1}"/>
     </xacro:unless>
     <xacro:macro name="robotiq_85_gripper" params="prefix parent *origin">
@@ -18,5 +24,5 @@
             <visual>
                 <geometry>
-                    <mesh filename="package://QR/movo_description_drake/meshes/manipulation/robotiq/visual/kinova_robotiq_coupler.dae"/>
+                    <mesh filename="package://QR/movo_description_drake/meshes/manipulation/robotiq/collision/kinova_robotiq_coupler.obj"/>
                 </geometry>
             </visual>
@@ -49,5 +55,5 @@
             <visual>
                 <geometry>
-                    <mesh filename="package://QR/movo_description_drake/meshes/manipulation/robotiq/visual/robotiq_85_base_link.dae"/>
+                    <mesh filename="package://QR/movo_description_drake/meshes/manipulation/robotiq/collision/robotiq_85_base_link.obj"/>
                 </geometry>
             </visual>
@@ -85,12 +91,14 @@
             <origin rpy="0.0 0.0 0.0" xyz="0.05490451627 -0.03060114443 0.0"/>
             <limit lower="-3.14" upper="3.14" velocity="100.0" effort="1000"/>
+            <xacro:unless value="$(optenv REPLACE_MIMIC false)">
             <xacro:unless value="$(optenv WELD_FINGERS false)">
               <mimic joint="${prefix}gripper_finger1_joint"/>
             </xacro:unless>
+            </xacro:unless>
         </joint>
         <link name="${prefix}gripper_finger1_knuckle_link">
             <visual>
                 <geometry>
-                    <mesh filename="package://QR/movo_description_drake/meshes/manipulation/robotiq/visual/robotiq_85_knuckle_link.dae"/>
+                    <mesh filename="package://QR/movo_description_drake/meshes/manipulation/robotiq/collision/robotiq_85_knuckle_link.obj"/>
                 </geometry>
             </visual>
@@ -118,5 +126,5 @@
             <visual>
                 <geometry>
-                    <mesh filename="package://QR/movo_description_drake/meshes/manipulation/robotiq/visual/robotiq_85_knuckle_link.dae"/>
+                    <mesh filename="package://QR/movo_description_drake/meshes/manipulation/robotiq/collision/robotiq_85_knuckle_link.obj"/>
                 </geometry>
             </visual>
@@ -154,5 +162,5 @@
             <visual>
                 <geometry>
-                    <mesh filename="package://QR/movo_description_drake/meshes/manipulation/robotiq/visual/robotiq_85_finger_link.dae"/>
+                    <mesh filename="package://QR/movo_description_drake/meshes/manipulation/robotiq/collision/robotiq_85_finger_link.obj"/>
                 </geometry>
             </visual>
@@ -180,5 +188,5 @@
             <visual>
                 <geometry>
-                    <mesh filename="package://QR/movo_description_drake/meshes/manipulation/robotiq/visual/robotiq_85_finger_link.dae"/>
+                    <mesh filename="package://QR/movo_description_drake/meshes/manipulation/robotiq/collision/robotiq_85_finger_link.obj"/>
                 </geometry>
             </visual>
@@ -203,4 +211,21 @@
             <kd>1.0</kd>
         </gazebo>
+        <xacro:if value="$(optenv REPLACE_MIMIC false)">
+          <joint name="${prefix}gripper_finger1_inner_knuckle_joint" type="revolute">
+              <parent link="${prefix}gripper_base_link"/>
+              <child link="${prefix}gripper_finger1_inner_knuckle_link"/>
+              <axis xyz="0 0 1"/>
+              <origin xyz="0.06142 0.0127 0" rpy="${M_PI} 0.0 0.0" />
+              <limit lower="-3.14" upper="3.14" velocity="100.0" effort="0.1"/>
+          </joint>
+          <joint name="${prefix}gripper_finger2_inner_knuckle_joint" type="revolute">
+              <parent link="${prefix}gripper_base_link"/>
+              <child link="${prefix}gripper_finger2_inner_knuckle_link"/>
+              <axis xyz="0 0 1"/>
+              <origin xyz="0.06142 -0.0127 0" rpy="0 0 0"/>
+              <limit lower="-3.14" upper="3.14" velocity="100.0" effort="0.1"/>
+          </joint>
+        </xacro:if>
+        <xacro:unless value="$(optenv REPLACE_MIMIC false)">
         <joint name="${prefix}gripper_finger1_inner_knuckle_joint" type="${revolute_or_fixed}">
             <parent link="${prefix}gripper_base_link"/>
@@ -209,6 +234,8 @@
             <origin xyz="0.06142 0.0127 0" rpy="${M_PI} 0.0 0.0" />
             <limit lower="-3.14" upper="3.14" velocity="100.0" effort="0.1"/>
+            <xacro:unless value="$(optenv REPLACE_MIMIC false)">
             <xacro:unless value="$(optenv WELD_FINGERS false)">
               <mimic joint="${prefix}gripper_finger1_joint" offset="0"/>
+            </xacro:unless>
             </xacro:unless>
         </joint>
@@ -219,12 +246,15 @@
             <origin xyz="0.06142 -0.0127 0" rpy="0 0 0"/>
             <limit lower="-3.14" upper="3.14" velocity="100.0" effort="0.1"/>
+            <xacro:unless value="$(optenv REPLACE_MIMIC false)">
             <xacro:unless value="$(optenv WELD_FINGERS false)">
               <mimic joint="${prefix}gripper_finger1_joint" offset="0"/>
             </xacro:unless>
-        </joint>
+            </xacro:unless>
+        </joint>
+        </xacro:unless>
         <link name="${prefix}gripper_finger1_inner_knuckle_link">
             <visual>
                 <geometry>
-                    <mesh filename="package://QR/movo_description_drake/meshes/manipulation/robotiq/visual/robotiq_85_inner_knuckle_link.dae"/>
+                    <mesh filename="package://QR/movo_description_drake/meshes/manipulation/robotiq/collision/robotiq_85_inner_knuckle_link.obj"/>
                 </geometry>
             </visual>
@@ -252,5 +282,5 @@
             <visual>
                 <geometry>
-                    <mesh filename="package://QR/movo_description_drake/meshes/manipulation/robotiq/visual/robotiq_85_inner_knuckle_link.dae"/>
+                    <mesh filename="package://QR/movo_description_drake/meshes/manipulation/robotiq/collision/robotiq_85_inner_knuckle_link.obj"/>
                 </geometry>
             </visual>
@@ -281,6 +311,8 @@
             <origin xyz="0.04303959807 -0.03759940821 0.0" rpy="0.0 0.0 0.0"/>
             <limit lower="-3.14" upper="3.14" velocity="100.0" effort="0.1"/>
+            <xacro:unless value="$(optenv REPLACE_MIMIC false)">
             <xacro:unless value="$(optenv WELD_FINGERS false)">
               <mimic joint="${prefix}gripper_finger1_joint" multiplier="-1"/>
+            </xacro:unless>
             </xacro:unless>
         </joint>
@@ -291,12 +323,14 @@
             <origin rpy="0.0 0.0 0.0" xyz="0.04303959807 -0.03759940821  0.0"/>
             <limit lower="-3.14" upper="3.14" velocity="100.0" effort="0.1"/>
+            <xacro:unless value="$(optenv REPLACE_MIMIC false)">
             <xacro:unless value="$(optenv WELD_FINGERS false)">
               <mimic joint="${prefix}gripper_finger1_joint" multiplier="-1"/>
             </xacro:unless>
+            </xacro:unless>
         </joint>
         <link name="${prefix}gripper_finger1_finger_tip_link">
             <visual>
                 <geometry>
-                    <mesh filename="package://QR/movo_description_drake/meshes/manipulation/robotiq/visual/robotiq_85_finger_tip_link.dae"/>
+                    <mesh filename="package://QR/movo_description_drake/meshes/manipulation/robotiq/collision/robotiq_85_finger_tip_link.obj"/>
                 </geometry>
             </visual>
@@ -324,5 +358,5 @@
             <visual>
                 <geometry>
-                    <mesh filename="package://QR/movo_description_drake/meshes/manipulation/robotiq/visual/robotiq_85_finger_tip_link.dae"/>
+                    <mesh filename="package://QR/movo_description_drake/meshes/manipulation/robotiq/collision/robotiq_85_finger_tip_link.obj"/>
                 </geometry>
             </visual>

File: movo_common/movo_description/urdf/movo_components/movo_base.urdf.xacro (robot description, xacro)
@@ -108,5 +108,5 @@
 				<origin xyz="0 0 0" rpy="0 0 0" />
 				<geometry>
-					<mesh filename="package://QR/movo_description_drake/meshes/movo_components/visual/vector_base.dae" />
+					<mesh filename="package://QR/movo_description_drake/meshes/movo_components/collision/vector_base_collision.obj" />
 				</geometry>
         <material>
@@ -144,5 +144,5 @@
 				<origin xyz="0 0 0" rpy="0 0 0" />
 				<geometry>
-					<mesh filename="package://QR/movo_description_drake/meshes/movo_components/visual/movo_fixed_payload.dae" />
+					<mesh filename="package://QR/movo_description_drake/meshes/movo_components/collision/movo_fixed_body_collision.obj" />
 				</geometry>
 			</visual>
@@ -162,5 +162,5 @@
 		    <visual>
 			    <geometry>
-				    <mesh filename="package://QR/movo_description_drake/meshes/movo_components/visual/movo_moving_payload.dae" />
+				    <mesh filename="package://QR/movo_description_drake/meshes/movo_components/collision/movo_upper_body_collision.obj" />
 			    </geometry>
 		    </visual>

File: movo_common/movo_description/urdf/movo_components/movo_body.urdf.xacro (robot description, xacro)
@@ -48,5 +48,5 @@
 				<origin xyz="0 0 0" rpy="0 0 0" />
 				<geometry>
-					<mesh filename="package://QR/movo_description_drake/meshes/movo_body/movo_lower_body.dae" />
+					<mesh filename="package://QR/movo_description_drake/meshes/movo_body/movo_lower_body.obj" />
 				</geometry>
         <material>
@@ -71,5 +71,5 @@
 				<origin xyz="0 0 0" rpy="0 0 0" />
 				<geometry>
-					<mesh filename="package://QR/movo_description_drake/meshes/movo_body/movo_upper_body.dae" />
+					<mesh filename="package://QR/movo_description_drake/meshes/movo_body/movo_upper_body.obj" />
 				</geometry>
         <material>
@@ -111,5 +111,5 @@
 				<origin xyz="0 0 0" rpy="0 0 0" />
 				<geometry>
-					<mesh filename="package://QR/movo_description_drake/meshes/movo_body/movo_mid_body.dae" />
+					<mesh filename="package://QR/movo_description_drake/meshes/movo_body/movo_mid_body.obj" />
 				</geometry>
         <material>

File: movo_common/movo_description/urdf/movo_components/movo_pan_tilt.urdf.xacro (robot description, xacro)
@@ -39,5 +39,5 @@
 			<visual>
 				<geometry>
-					<mesh filename="package://QR/movo_description_drake/meshes/pan_tilt/visual/pan_tilt_base.dae" />
+					<mesh filename="package://QR/movo_description_drake/meshes/pan_tilt/collision/pan_tilt_base.obj" />
 				</geometry>
         <material>
@@ -77,5 +77,5 @@
 			<visual>
 				<geometry>
-					<mesh filename="package://QR/movo_description_drake/meshes/pan_tilt/visual/pan_link.dae" />
+					<mesh filename="package://QR/movo_description_drake/meshes/pan_tilt/collision/pan_link.obj" />
 				</geometry>
         <material>
@@ -116,5 +116,5 @@
 			<visual>
 				<geometry>
-					<mesh filename="package://QR/movo_description_drake/meshes/pan_tilt/visual/tilt_link.dae" />
+					<mesh filename="package://QR/movo_description_drake/meshes/pan_tilt/collision/tilt_link.obj" />
 				</geometry>
         <material>

File: movo_common/movo_description/urdf/movo_components/proto2_arm_mount.urdf.xacro (robot description, xacro)
@@ -42,5 +42,5 @@
 			<collision>
 				<geometry>
-					<mesh filename="package://QR/movo_description_drake/meshes/proto2/collision/proto2_arm_mount_collision.obj" />
+					<mesh filename="package://QR/movo_description_drake/meshes/proto2/collision/proto2_arm_mount_collision.dae" />
 				</geometry>
 			</collision>

File: movo_common/movo_description/urdf/movo_components/proto2_base.urdf.xacro (robot description, xacro)
@@ -51,5 +51,5 @@
             <collision>
 				<geometry>
-					<mesh filename="package://QR/movo_description_drake/meshes/proto2/collision/proto2_base_collision.obj" />
+					<mesh filename="package://QR/movo_description_drake/meshes/proto2/collision/proto2_base_collision.dae" />
 				</geometry>
 			</collision>

File: movo_common/movo_description/urdf/movo_components/proto2_frame.urdf.xacro (robot description, xacro)
@@ -42,5 +42,5 @@
 			<collision>
 				<geometry>
-					<mesh filename="package://QR/movo_description_drake/meshes/proto2/collision/proto2_frame_collision.obj" />
+					<mesh filename="package://QR/movo_description_drake/meshes/proto2/collision/proto2_frame_collision.dae" />
 				</geometry>
 			</collision>

File: movo_common/movo_description/urdf/sensors/kinect_one_sensor.urdf.xacro (robot description, xacro)
@@ -57,5 +57,5 @@
 			<visual>
 				<geometry>
-					<mesh filename="package://QR/movo_description_drake/meshes/sensors/visual/kinect_one.dae" />
+					<mesh filename="package://QR/movo_description_drake/meshes/sensors/collision/kinect_one_collision.obj" />
 				</geometry>
         <material>

File: movo_common/movo_description/urdf/sensors/sick_tim.urdf.xacro (robot description, xacro)
@@ -35,9 +35,9 @@
         </joint>
         <link name="${laser_prefix}_laser_link">
-            <visual>
+<!--            <visual>
                 <geometry>
-                    <mesh filename="package://QR/movo_description_drake/meshes/sensors/visual/sick_tim.dae" />
+                    <mesh filename="package://QR/movo_description_drake/meshes/sensors/collision/sick_tim.dae" />
                 </geometry>
-            </visual>
+            </visual> -->
             <collision>
                 <geometry>
