Commit message: both robotiq models parse (stand-alone) into Drake
though I'm missing some .mtl files for the woven model.

File: movo_common/movo_description/urdf/manipulation/robotiq/robotiq_85_gripper.urdf (robot description, URDF)
Before this commit: robot robotiq_85_gripper, 0 links, 0 joints
Links:
- added link gripper_base_link, mass 0.636951; collision mesh filename=package://movo_description/meshes/manipulation/robotiq/coll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; visual mesh filename=package://movo_description/meshes/manipulation/robotiq/visu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
- added link gripper_finger1_finger_link, mass 0.027309; collision mesh filename=package://movo_description/meshes/manipulation/robotiq/coll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; visual mesh filename=package://movo_description/meshes/manipulation/robotiq/visu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
- added link gripper_finger1_finger_tip_link, mass 0.019555; collision sphere radius=1e-7; collision sphere radius=1e-7
- added link gripper_finger1_inner_knuckle_link, mass 0.029951; visual mesh filename=package://movo_description/meshes/manipulation/robotiq/visu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
- added link gripper_finger1_knuckle_link, mass 0.018491; collision mesh filename=package://movo_description/meshes/manipulation/robotiq/coll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; visual mesh filename=package://movo_description/meshes/manipulation/robotiq/visu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
- added link gripper_finger2_finger_link, mass 0.027309; collision mesh filename=package://movo_description/meshes/manipulation/robotiq/coll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; visual mesh filename=package://movo_description/meshes/manipulation/robotiq/visu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
- added link gripper_finger2_finger_tip_link, mass 0.019555; collision box size=0.0375 0.00675 0.022; visual mesh filename=package://movo_description/meshes/manipulation/robotiq/visu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
- added link gripper_finger2_inner_knuckle_link, mass 0.029951; visual mesh filename=package://movo_description/meshes/manipulation/robotiq/visu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
- added link gripper_finger2_knuckle_link, mass 0.018491; collision mesh filename=package://movo_description/meshes/manipulation/robotiq/coll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; visual mesh filename=package://movo_description/meshes/manipulation/robotiq/visu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
- added link robotiq_coupler_link, mass 0.1; collision mesh filename=package://movo_description/meshes/manipulation/robotiq/coll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; visual mesh filename=package://movo_description/meshes/manipulation/robotiq/visu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
Joints:
- added joint gripper_base_joint: type fixed, parent robotiq_coupler_link, child gripper_base_link, origin xyz=0 0 -0.05105 rpy=-1.570795 1.570795 0.0
- added joint gripper_finger1_finger_joint: type fixed, parent gripper_finger1_knuckle_link, child gripper_finger1_finger_link, origin xyz=-0.00408552455 -0.03148604435 0.0 rpy=0 0 0
- added joint gripper_finger1_finger_tip_joint: type revolute, parent gripper_finger1_inner_knuckle_link, child gripper_finger1_finger_tip_link, origin xyz=0.04303959807 -0.03759940821 0.0 rpy=0.0 0.0 0.0, axis 0 0 1, limit lower=-3.14 upper=3.14 effort=0.1 velocity=100.0, mimic joint=gripper_finger1_joint multiplier=-1
- added joint gripper_finger1_inner_knuckle_joint: type revolute, parent gripper_base_link, child gripper_finger1_inner_knuckle_link, origin xyz=0.06142 0.0127 0 rpy=3.14159 0.0 0.0, axis 0 0 1, limit lower=-3.14 upper=3.14 effort=0.1 velocity=100.0, mimic joint=gripper_finger1_joint offset=0
- added joint gripper_finger1_joint: type revolute, parent gripper_base_link, child gripper_finger1_knuckle_link, origin xyz=0.05490451627 0.03060114443 0.0 rpy=3.14159 0.0 0.0, axis 0 0 1, limit lower=0.0 upper=0.804 effort=1000 velocity=2.0
- added joint gripper_finger2_finger_joint: type fixed, parent gripper_finger2_knuckle_link, child gripper_finger2_finger_link, origin xyz=-0.00408552455 -0.03148604435 0.0 rpy=0 0 0
- added joint gripper_finger2_finger_tip_joint: type revolute, parent gripper_finger2_inner_knuckle_link, child gripper_finger2_finger_tip_link, origin xyz=0.04303959807 -0.03759940821  0.0 rpy=0.0 0.0 0.0, axis 0 0 1, limit lower=-3.14 upper=3.14 effort=0.1 velocity=100.0, mimic joint=gripper_finger1_joint multiplier=-1
- added joint gripper_finger2_inner_knuckle_joint: type revolute, parent gripper_base_link, child gripper_finger2_inner_knuckle_link, origin xyz=0.06142 -0.0127 0 rpy=0 0 0, axis 0 0 1, limit lower=-3.14 upper=3.14 effort=0.1 velocity=100.0, mimic joint=gripper_finger1_joint offset=0
- added joint gripper_finger2_joint: type revolute, parent gripper_base_link, child gripper_finger2_knuckle_link, origin xyz=0.05490451627 -0.03060114443 0.0 rpy=0.0 0.0 0.0, axis 0 0 1, limit lower=-3.14 upper=3.14 effort=1000 velocity=100.0, mimic joint=gripper_finger1_joint

File: movo_common/movo_description/urdf/manipulation/robotiq/robotiq_85_gripper.urdf.xacro (robot description, xacro)
@@ -16,18 +16,20 @@
     </xacro:unless>
     <xacro:macro name="robotiq_85_gripper" params="prefix parent *origin">
-        <joint name="${prefix}kinova_robotiq_coupler_joint" type="fixed">
-            <parent link="${parent}"/>
-            <child link="${prefix}robotiq_coupler_link"/>
-            <xacro:insert_block name="origin"/>
-        </joint>
+        <xacro:if value="${parent != ''}">
+          <joint name="${prefix}kinova_robotiq_coupler_joint" type="fixed">
+              <parent link="${parent}"/>
+              <child link="${prefix}robotiq_coupler_link"/>
+              <xacro:insert_block name="origin"/>
+          </joint>
+        </xacro:if>
         <link name="${prefix}robotiq_coupler_link">
             <visual>
                 <geometry>
-                    <mesh filename="package://QR/movo_description_drake/meshes/manipulation/robotiq/visual/kinova_robotiq_coupler.obj"/>
-                </geometry>
-            </visual>
-            <collision>
-                <geometry>
-                    <mesh filename="package://QR/movo_description_drake/meshes/manipulation/robotiq/collision/kinova_robotiq_coupler.obj"/>
+                    <mesh filename="package://movo_description/meshes/manipulation/robotiq/visual/kinova_robotiq_coupler.obj"/>
+                </geometry>
+            </visual>
+            <collision>
+                <geometry>
+                    <mesh filename="package://movo_description/meshes/manipulation/robotiq/collision/kinova_robotiq_coupler.obj"/>
                 </geometry>
             </collision>
@@ -55,10 +57,10 @@
             <visual>
                 <geometry>
-                    <mesh filename="package://QR/movo_description_drake/meshes/manipulation/robotiq/visual/robotiq_85_base_link.obj"/>
-                </geometry>
-            </visual>
-            <collision>
-                <geometry>
-                    <mesh filename="package://QR/movo_description_drake/meshes/manipulation/robotiq/collision/robotiq_85_base_link.obj"/>
+                    <mesh filename="package://movo_description/meshes/manipulation/robotiq/visual/robotiq_85_base_link.obj"/>
+                </geometry>
+            </visual>
+            <collision>
+                <geometry>
+                    <mesh filename="package://movo_description/meshes/manipulation/robotiq/collision/robotiq_85_base_link.obj"/>
                 </geometry>
             </collision>
@@ -100,10 +102,10 @@
             <visual>
                 <geometry>
-                    <mesh filename="package://QR/movo_description_drake/meshes/manipulation/robotiq/visual/robotiq_85_knuckle_link.obj"/>
-                </geometry>
-            </visual>
-            <collision>
-                <geometry>
-                    <mesh filename="package://QR/movo_description_drake/meshes/manipulation/robotiq/collision/robotiq_85_knuckle_link.obj"/>
+                    <mesh filename="package://movo_description/meshes/manipulation/robotiq/visual/robotiq_85_knuckle_link.obj"/>
+                </geometry>
+            </visual>
+            <collision>
+                <geometry>
+                    <mesh filename="package://movo_description/meshes/manipulation/robotiq/collision/robotiq_85_knuckle_link.obj"/>
                 </geometry>
             </collision>
@@ -126,10 +128,10 @@
             <visual>
                 <geometry>
-                    <mesh filename="package://QR/movo_description_drake/meshes/manipulation/robotiq/visual/robotiq_85_knuckle_link.obj"/>
-                </geometry>
-            </visual>
-            <collision>
-                <geometry>
-                    <mesh filename="package://QR/movo_description_drake/meshes/manipulation/robotiq/collision/robotiq_85_knuckle_link.obj"/>
+                    <mesh filename="package://movo_description/meshes/manipulation/robotiq/visual/robotiq_85_knuckle_link.obj"/>
+                </geometry>
+            </visual>
+            <collision>
+                <geometry>
+                    <mesh filename="package://movo_description/meshes/manipulation/robotiq/collision/robotiq_85_knuckle_link.obj"/>
                 </geometry>
             </collision>
@@ -162,10 +164,10 @@
             <visual>
                 <geometry>
-                    <mesh filename="package://QR/movo_description_drake/meshes/manipulation/robotiq/visual/robotiq_85_finger_link.obj"/>
-                </geometry>
-            </visual>
-            <collision>
-                <geometry>
-                    <mesh filename="package://QR/movo_description_drake/meshes/manipulation/robotiq/collision/robotiq_85_finger_link.obj"/>
+                    <mesh filename="package://movo_description/meshes/manipulation/robotiq/visual/robotiq_85_finger_link.obj"/>
+                </geometry>
+            </visual>
+            <collision>
+                <geometry>
+                    <mesh filename="package://movo_description/meshes/manipulation/robotiq/collision/robotiq_85_finger_link.obj"/>
                 </geometry>
             </collision>
@@ -188,10 +190,10 @@
             <visual>
                 <geometry>
-                    <mesh filename="package://QR/movo_description_drake/meshes/manipulation/robotiq/visual/robotiq_85_finger_link.obj"/>
-                </geometry>
-            </visual>
-            <collision>
-                <geometry>
-                    <mesh filename="package://QR/movo_description_drake/meshes/manipulation/robotiq/collision/robotiq_85_finger_link.obj"/>
+                    <mesh filename="package://movo_description/meshes/manipulation/robotiq/visual/robotiq_85_finger_link.obj"/>
+                </geometry>
+            </visual>
+            <collision>
+                <geometry>
+                    <mesh filename="package://movo_description/meshes/manipulation/robotiq/collision/robotiq_85_finger_link.obj"/>
                 </geometry>
             </collision>
@@ -256,5 +258,5 @@
             <visual>
                 <geometry>
-                    <mesh filename="package://QR/movo_description_drake/meshes/manipulation/robotiq/visual/robotiq_85_inner_knuckle_link.obj"/>
+                    <mesh filename="package://movo_description/meshes/manipulation/robotiq/visual/robotiq_85_inner_knuckle_link.obj"/>
                 </geometry>
             </visual>
@@ -262,5 +264,5 @@
             <collision>
                 <geometry>
-                    <mesh filename="package://QR/movo_description_drake/meshes/manipulation/robotiq/collision/robotiq_85_inner_knuckle_link.obj"/>
+                    <mesh filename="package://movo_description/meshes/manipulation/robotiq/collision/robotiq_85_inner_knuckle_link.obj"/>
                 </geometry>
             </collision>
@@ -284,5 +286,5 @@
             <visual>
                 <geometry>
-                    <mesh filename="package://QR/movo_description_drake/meshes/manipulation/robotiq/visual/robotiq_85_inner_knuckle_link.obj"/>
+                    <mesh filename="package://movo_description/meshes/manipulation/robotiq/visual/robotiq_85_inner_knuckle_link.obj"/>
                 </geometry>
             </visual>
@@ -290,5 +292,5 @@
             <collision>
                 <geometry>
-                    <mesh filename="package://QR/movo_description_drake/meshes/manipulation/robotiq/collision/robotiq_85_inner_knuckle_link.obj"/>
+                    <mesh filename="package://movo_description/meshes/manipulation/robotiq/collision/robotiq_85_inner_knuckle_link.obj"/>
                 </geometry>
             </collision>
@@ -336,5 +338,5 @@
             <visual>
                 <geometry>
-                    <mesh filename="package://QR/movo_description_drake/meshes/manipulation/robotiq/visual/robotiq_85_finger_tip_link.obj"/>
+                    <mesh filename="package://movo_description/meshes/manipulation/robotiq/visual/robotiq_85_finger_tip_link.obj"/>
                 </geometry>
             </visual>
@@ -418,5 +420,5 @@
             <visual>
                 <geometry>
-                    <mesh filename="package://QR/movo_description_drake/meshes/manipulation/robotiq/visual/robotiq_85_finger_tip_link.obj"/>
+                    <mesh filename="package://movo_description/meshes/manipulation/robotiq/visual/robotiq_85_finger_tip_link.obj"/>
                 </geometry>
             </visual>
@@ -429,5 +431,5 @@
                 <!--
                 <geometry>
-                    <mesh filename="package://QR/movo_description_drake/meshes/manipulation/robotiq/collision/robotiq_85_finger_tip_link.obj"/>
+                    <mesh filename="package://movo_description/meshes/manipulation/robotiq/collision/robotiq_85_finger_tip_link.obj"/>
                 </geometry>
               -->
@@ -449,4 +451,5 @@
         </gazebo>
         <xacro:robotiq_85_gripper_transmission prefix="${prefix}" />
+        <xacro:if value="${parent != ''}">
         <drake:collision_filter_group name="${prefix}link_6_coupler">
           <!-- <drake:member link="${prefix}link_6" /> -->
@@ -456,4 +459,5 @@
           <drake:ignored_collision_filter_group name="${prefix}link_6_coupler" />
         </drake:collision_filter_group>
+        </xacro:if>
         <drake:collision_filter_group name="${prefix}finger_1">
           <drake:member link="${prefix}gripper_finger1_finger_link" />
