Commit message: fixup robotiq and movo geometry

File: movo_common/movo_description/urdf/manipulation/robotiq/robotiq_85_gripper.urdf.xacro (robot description, xacro)
@@ -24,5 +24,5 @@
             <visual>
                 <geometry>
-                    <mesh filename="package://QR/movo_description_drake/meshes/manipulation/robotiq/collision/kinova_robotiq_coupler.obj"/>
+                    <mesh filename="package://QR/movo_description_drake/meshes/manipulation/robotiq/visual/kinova_robotiq_coupler.obj"/>
                 </geometry>
             </visual>
@@ -55,5 +55,5 @@
             <visual>
                 <geometry>
-                    <mesh filename="package://QR/movo_description_drake/meshes/manipulation/robotiq/collision/robotiq_85_base_link.obj"/>
+                    <mesh filename="package://QR/movo_description_drake/meshes/manipulation/robotiq/visual/robotiq_85_base_link.obj"/>
                 </geometry>
             </visual>
@@ -100,5 +100,5 @@
             <visual>
                 <geometry>
-                    <mesh filename="package://QR/movo_description_drake/meshes/manipulation/robotiq/collision/robotiq_85_knuckle_link.obj"/>
+                    <mesh filename="package://QR/movo_description_drake/meshes/manipulation/robotiq/visual/robotiq_85_knuckle_link.obj"/>
                 </geometry>
             </visual>
@@ -126,5 +126,5 @@
             <visual>
                 <geometry>
-                    <mesh filename="package://QR/movo_description_drake/meshes/manipulation/robotiq/collision/robotiq_85_knuckle_link.obj"/>
+                    <mesh filename="package://QR/movo_description_drake/meshes/manipulation/robotiq/visual/robotiq_85_knuckle_link.obj"/>
                 </geometry>
             </visual>
@@ -162,5 +162,5 @@
             <visual>
                 <geometry>
-                    <mesh filename="package://QR/movo_description_drake/meshes/manipulation/robotiq/collision/robotiq_85_finger_link.obj"/>
+                    <mesh filename="package://QR/movo_description_drake/meshes/manipulation/robotiq/visual/robotiq_85_finger_link.obj"/>
                 </geometry>
             </visual>
@@ -188,5 +188,5 @@
             <visual>
                 <geometry>
-                    <mesh filename="package://QR/movo_description_drake/meshes/manipulation/robotiq/collision/robotiq_85_finger_link.obj"/>
+                    <mesh filename="package://QR/movo_description_drake/meshes/manipulation/robotiq/visual/robotiq_85_finger_link.obj"/>
                 </geometry>
             </visual>
@@ -256,5 +256,5 @@
             <visual>
                 <geometry>
-                    <mesh filename="package://QR/movo_description_drake/meshes/manipulation/robotiq/collision/robotiq_85_inner_knuckle_link.obj"/>
+                    <mesh filename="package://QR/movo_description_drake/meshes/manipulation/robotiq/visual/robotiq_85_inner_knuckle_link.obj"/>
                 </geometry>
             </visual>
@@ -282,5 +282,5 @@
             <visual>
                 <geometry>
-                    <mesh filename="package://QR/movo_description_drake/meshes/manipulation/robotiq/collision/robotiq_85_inner_knuckle_link.obj"/>
+                    <mesh filename="package://QR/movo_description_drake/meshes/manipulation/robotiq/visual/robotiq_85_inner_knuckle_link.obj"/>
                 </geometry>
             </visual>
@@ -332,5 +332,5 @@
             <visual>
                 <geometry>
-                    <mesh filename="package://QR/movo_description_drake/meshes/manipulation/robotiq/collision/robotiq_85_finger_tip_link.obj"/>
+                    <mesh filename="package://QR/movo_description_drake/meshes/manipulation/robotiq/visual/robotiq_85_finger_tip_link.obj"/>
                 </geometry>
             </visual>
@@ -358,5 +358,5 @@
             <visual>
                 <geometry>
-                    <mesh filename="package://QR/movo_description_drake/meshes/manipulation/robotiq/collision/robotiq_85_finger_tip_link.obj"/>
+                    <mesh filename="package://QR/movo_description_drake/meshes/manipulation/robotiq/visual/robotiq_85_finger_tip_link.obj"/>
                 </geometry>
             </visual>

File: movo_common/movo_description/urdf/movo_components/movo_base.urdf.xacro (robot description, xacro)
@@ -140,5 +140,4 @@
 				</geometry>
 			</collision>
-      -->
 			<visual>
 				<origin xyz="0 0 0" rpy="0 0 0" />
@@ -147,4 +146,5 @@
 				</geometry>
 			</visual>
+      -->
 		</link>
 		<gazebo reference="linear_actuator_fixed_link">
@@ -160,9 +160,10 @@
         </joint>
         <link name="linear_actuator_link">
+        <!--
 		    <visual>
 			    <geometry>
 				    <mesh filename="package://QR/movo_description_drake/meshes/movo_components/collision/movo_upper_body_collision.obj" />
 			    </geometry>
-		    </visual>
+		    </visual>-->
         <!-- russt: removed this because it was causing self-collisions
 		    <collision>

Commit message: add world link; simple gripper finger tip geometry

File: movo_common/movo_description/urdf/manipulation/robotiq/robotiq_85_gripper.urdf.xacro (robot description, xacro)
@@ -336,7 +336,14 @@
             </visual>
             <collision>
+                <!-- box for finger tip computed by measuring in blender -->
+                <origin xyz="0.02575 0.004375 0" />
+                <geometry>
+                    <box size="0.0375 0.00675 0.022" />
+                </geometry>
+                <!--
                 <geometry>
                     <mesh filename="package://QR/movo_description_drake/meshes/manipulation/robotiq/collision/robotiq_85_finger_tip_link.obj"/>
                 </geometry>
+              -->
             </collision>
             <inertial>
@@ -362,7 +369,14 @@
             </visual>
             <collision>
+                <!-- box for finger tip computed by measuring in blender -->
+                <origin xyz="0.02575 0.004375 0" />
+                <geometry>
+                    <box size="0.0375 0.00675 0.022" />
+                </geometry>
+                <!--
                 <geometry>
                     <mesh filename="package://QR/movo_description_drake/meshes/manipulation/robotiq/collision/robotiq_85_finger_tip_link.obj"/>
                 </geometry>
+              -->
             </collision>
             <inertial>

File: movo_common/movo_description/urdf/movo_components/movo_base.urdf.xacro (robot description, xacro)
@@ -34,4 +34,5 @@
 	  <xacro:macro name="movo_base">
         <!-- russt: added an actuated planar joint to the base. -->
+        <link name="world"/>
         <link name="base_link_0"/>
         <link name="base_link_1"/>

Commit message: add contact spheres until I enable hydro

File: movo_common/movo_description/urdf/manipulation/robotiq/robotiq_85_gripper.urdf.xacro (robot description, xacro)
@@ -259,4 +259,5 @@
                 </geometry>
             </visual>
+            <!--
             <collision>
                 <geometry>
@@ -264,4 +265,5 @@
                 </geometry>
             </collision>
+            -->
             <inertial>
                 <mass value="0.029951" />
@@ -285,4 +287,5 @@
                 </geometry>
             </visual>
+            <!--
             <collision>
                 <geometry>
@@ -290,4 +293,5 @@
                 </geometry>
             </collision>
+            -->
             <inertial>
                 <mass value="0.029951" />
@@ -339,5 +343,8 @@
                 <origin xyz="0.02575 0.004375 0" />
                 <geometry>
+                    <!--
                     <box size="0.0375 0.00675 0.022" />
+                    -->
+                    <box size="0.037 0.00625 0.0215" />
                 </geometry>
                 <!--
@@ -346,4 +353,65 @@
                 </geometry>
               -->
+            </collision>
+            <!-- manually add spheres until hydroelastic is enabled -->
+            <collision>
+              <origin xyz="0.007 0.00775 0.011" />
+              <geometry>
+                <sphere radius="1e-7" />
+              </geometry>
+            </collision>
+            <collision>
+              <origin xyz="0.016375 0.00775 0.011" />
+              <geometry>
+                <sphere radius="1e-7" />
+              </geometry>
+            </collision>
+            <collision>
+              <origin xyz="0.02575 0.00775 0.011" />
+              <geometry>
+                <sphere radius="1e-7" />
+              </geometry>
+            </collision>
+            <collision>
+              <origin xyz="0.035125 0.00775 0.011" />
+              <geometry>
+                <sphere radius="1e-7" />
+              </geometry>
+            </collision>
+            <collision>
+              <origin xyz="0.0445 0.00775 0.011" />
+              <geometry>
+                <sphere radius="1e-7" />
+              </geometry>
+            </collision>
+            <collision>
+              <origin xyz="0.007 0.00775 -0.011" />
+              <geometry>
+                <sphere radius="1e-7" />
+              </geometry>
+            </collision>
+            <collision>
+              <origin xyz="0.016375 0.00775 -0.011" />
+              <geometry>
+                <sphere radius="1e-7" />
+              </geometry>
+            </collision>
+            <collision>
+              <origin xyz="0.02575 0.00775 -0.011" />
+              <geometry>
+                <sphere radius="1e-7" />
+              </geometry>
+            </collision>
+            <collision>
+              <origin xyz="0.035125 0.00775 -0.011" />
+              <geometry>
+                <sphere radius="1e-7" />
+              </geometry>
+            </collision>
+            <collision>
+              <origin xyz="0.0445 0.00775 -0.011" />
+              <geometry>
+                <sphere radius="1e-7" />
+              </geometry>
             </collision>
             <inertial>

Commit message: Add movo obj files and sdf from woven

File: movo_common/movo_description/urdf/manipulation/robotiq/robotiq_85_gripper.urdf.xacro (robot description, xacro)
@@ -339,19 +339,4 @@
                 </geometry>
             </visual>
-            <collision>
-                <!-- box for finger tip computed by measuring in blender -->
-                <origin xyz="0.02575 0.004375 0" />
-                <geometry>
-                    <!--
-                    <box size="0.0375 0.00675 0.022" />
-                    -->
-                    <box size="0.037 0.00625 0.0215" />
-                </geometry>
-                <!--
-                <geometry>
-                    <mesh filename="package://QR/movo_description_drake/meshes/manipulation/robotiq/collision/robotiq_85_finger_tip_link.obj"/>
-                </geometry>
-              -->
-            </collision>
             <!-- manually add spheres until hydroelastic is enabled -->
             <collision>

Commit message: update robotiq xacro (not just urdf)

File: movo_common/movo_description/urdf/manipulation/robotiq/robotiq_85_gripper.urdf.xacro (robot description, xacro)
@@ -341,64 +341,22 @@
                 </geometry>
             </visual>
-            <!-- manually add spheres until hydroelastic is enabled -->
-            <collision>
-              <origin xyz="0.007 0.00775 0.011" />
-              <geometry>
-                <sphere radius="1e-7" />
-              </geometry>
-            </collision>
-            <collision>
-              <origin xyz="0.016375 0.00775 0.011" />
-              <geometry>
-                <sphere radius="1e-7" />
-              </geometry>
-            </collision>
-            <collision>
-              <origin xyz="0.02575 0.00775 0.011" />
-              <geometry>
-                <sphere radius="1e-7" />
-              </geometry>
-            </collision>
-            <collision>
-              <origin xyz="0.035125 0.00775 0.011" />
-              <geometry>
-                <sphere radius="1e-7" />
-              </geometry>
-            </collision>
-            <collision>
-              <origin xyz="0.0445 0.00775 0.011" />
-              <geometry>
-                <sphere radius="1e-7" />
-              </geometry>
-            </collision>
-            <collision>
-              <origin xyz="0.007 0.00775 -0.011" />
-              <geometry>
-                <sphere radius="1e-7" />
-              </geometry>
-            </collision>
-            <collision>
-              <origin xyz="0.016375 0.00775 -0.011" />
-              <geometry>
-                <sphere radius="1e-7" />
-              </geometry>
-            </collision>
-            <collision>
-              <origin xyz="0.02575 0.00775 -0.011" />
-              <geometry>
-                <sphere radius="1e-7" />
-              </geometry>
-            </collision>
-            <collision>
-              <origin xyz="0.035125 0.00775 -0.011" />
-              <geometry>
-                <sphere radius="1e-7" />
-              </geometry>
-            </collision>
-            <collision>
-              <origin xyz="0.0445 0.00775 -0.011" />
-              <geometry>
-                <sphere radius="1e-7" />
-              </geometry>
+            <collision>
+                <!-- box for finger tip computed by measuring in blender -->
+                <origin xyz="0.02575 0.004375 0"/>
+                <geometry>
+                    <box size="0.0375 0.00675 0.022"/>
+                </geometry>
+                <drake:proximity_properties>
+                    <drake:mu_static value="1.0"/>
+                    <drake:mu_dynamic value="1.0"/>
+                    <drake:hydroelastic_modulus value="1.0e5"/>
+                    <drake:hunt_crossley_dissipation value="10.0"/>
+                    <drake:compliant_hydroelastic/>
+                </drake:proximity_properties>
+                <!--
+                  <geometry>
+                      <mesh filename="package://movo_description/meshes/manipulation/robotiq/collision/robotiq_85_finger_tip_link.obj"/>
+                  </geometry>
+                -->
             </collision>
             <inertial>
@@ -425,13 +383,20 @@
             <collision>
                 <!-- box for finger tip computed by measuring in blender -->
-                <origin xyz="0.02575 0.004375 0" />
-                <geometry>
-                    <box size="0.0375 0.00675 0.022" />
-                </geometry>
+                <origin xyz="0.02575 0.004375 0"/>
+                <geometry>
+                    <box size="0.0375 0.00675 0.022"/>
+                </geometry>
+                <drake:proximity_properties>
+                    <drake:mu_static value="1.0"/>
+                    <drake:mu_dynamic value="1.0"/>
+                    <drake:hydroelastic_modulus value="1.0e5"/>
+                    <drake:hunt_crossley_dissipation value="10.0"/>
+                    <drake:compliant_hydroelastic/>
+                </drake:proximity_properties>
                 <!--
-                <geometry>
-                    <mesh filename="package://movo_description/meshes/manipulation/robotiq/collision/robotiq_85_finger_tip_link.obj"/>
-                </geometry>
-              -->
+                  <geometry>
+                      <mesh filename="package://movo_description/meshes/manipulation/robotiq/collision/robotiq_85_finger_tip_link.obj"/>
+                  </geometry>
+                -->
             </collision>
             <inertial>
