Commit message: re-enable mimic for torso

File: movo_common/movo_description/urdf/movo_components/movo_body.urdf.xacro (robot description, xacro)
@@ -31,4 +31,10 @@
     <xacro:property name="wheel_radius" value="0.0762" />
     <xacro:property name="M_PI" value="3.14159"/>
+    <xacro:if value="$(optenv WELD_FINGERS false)">
+      <xacro:property name="prismatic_or_fixed" value="fixed"/>
+    </xacro:if>
+    <xacro:unless value="$(optenv WELD_FINGERS false)">
+      <xacro:property name="prismatic_or_fixed" value="prismatic"/>
+    </xacro:unless>
 	<xacro:macro name="movo_body">
         <joint name="lower_body_joint" type="fixed">
@@ -78,8 +84,5 @@
 			</visual>
 		</link>
-        <!-- russt: make this fixed for now; it was causing problems with the inverse dynamics controllers.
-        <joint name="mid_body_joint" type="prismatic">
-        -->
-        <joint name="mid_body_joint" type="fixed">
+        <joint name="mid_body_joint" type="${prismatic_or_fixed}">
             <parent link="base_chassis_link" />
             <child link = "mid_body_link" />
@@ -88,5 +91,7 @@
             <limit lower="0.0" upper="0.2545608" effort="1000" velocity="0.20"/>
             <dynamics damping="0.0" friction="0.0"/>
-            <!-- <mimic joint="linear_joint" multiplier="0.5" offset="0.0" /> -->
+            <xacro:unless value="$(optenv WELD_FINGERS false)">
+              <mimic joint="linear_joint" multiplier="0.5" offset="0.0" />
+            </xacro:unless>
         </joint>
         <!-- russt: add transmission to avoid mimic joint
