Commit message: add black color as hotfix for missing textures

File: movo_common/movo_description/urdf/movo_components/movo_base.urdf.xacro (robot description, xacro)
@@ -110,4 +110,7 @@
 					<mesh filename="package://QR/movo_description_drake/meshes/movo_components/visual/vector_base.dae" />
 				</geometry>
+        <material>
+          <color rgba="0.1788232 0.1788232 0.1788232 1"/>
+        </material>
 			</visual>
 		</link>

File: movo_common/movo_description/urdf/movo_components/movo_body.urdf.xacro (robot description, xacro)
@@ -50,4 +50,7 @@
 					<mesh filename="package://QR/movo_description_drake/meshes/movo_body/movo_lower_body.dae" />
 				</geometry>
+        <material>
+          <color rgba="0.1788232 0.1788232 0.1788232 1"/>
+        </material>
 			</visual>
 		</link>
@@ -70,4 +73,7 @@
 					<mesh filename="package://QR/movo_description_drake/meshes/movo_body/movo_upper_body.dae" />
 				</geometry>
+        <material>
+          <color rgba="0.1788232 0.1788232 0.1788232 1"/>
+        </material>
 			</visual>
 		</link>
@@ -107,4 +113,7 @@
 					<mesh filename="package://QR/movo_description_drake/meshes/movo_body/movo_mid_body.dae" />
 				</geometry>
+        <material>
+          <color rgba="0.1788232 0.1788232 0.1788232 1"/>
+        </material>
 			</visual>
 		</link>

File: movo_common/movo_description/urdf/movo_components/movo_pan_tilt.urdf.xacro (robot description, xacro)
@@ -41,4 +41,7 @@
 					<mesh filename="package://QR/movo_description_drake/meshes/pan_tilt/visual/pan_tilt_base.dae" />
 				</geometry>
+        <material>
+          <color rgba="0.1788232 0.1788232 0.1788232 1"/>
+        </material>
 			</visual>
 			<collision>
@@ -76,4 +79,7 @@
 					<mesh filename="package://QR/movo_description_drake/meshes/pan_tilt/visual/pan_link.dae" />
 				</geometry>
+        <material>
+          <color rgba="0.1788232 0.1788232 0.1788232 1"/>
+        </material>
 			</visual>
 			<collision>
@@ -112,4 +118,7 @@
 					<mesh filename="package://QR/movo_description_drake/meshes/pan_tilt/visual/tilt_link.dae" />
 				</geometry>
+        <material>
+          <color rgba="0.1788232 0.1788232 0.1788232 1"/>
+        </material>
 			</visual>
 			<collision>

File: movo_common/movo_description/urdf/sensors/kinect_one_sensor.urdf.xacro (robot description, xacro)
@@ -59,4 +59,7 @@
 					<mesh filename="package://QR/movo_description_drake/meshes/sensors/visual/kinect_one.dae" />
 				</geometry>
+        <material>
+          <color rgba="0.1788232 0.1788232 0.1788232 1"/>
+        </material>
 			</visual>
 			<collision>

Commit message: switch back to visual geometry

File: movo_common/movo_description/urdf/movo_components/movo_base.urdf.xacro (robot description, xacro)
@@ -108,5 +108,5 @@
 				<origin xyz="0 0 0" rpy="0 0 0" />
 				<geometry>
-					<mesh filename="package://QR/movo_description_drake/meshes/movo_components/collision/vector_base_collision.obj" />
+					<mesh filename="package://QR/movo_description_drake/meshes/movo_components/visual/vector_base.obj" />
 				</geometry>
         <material>

File: movo_common/movo_description/urdf/movo_components/movo_pan_tilt.urdf.xacro (robot description, xacro)
@@ -39,5 +39,5 @@
 			<visual>
 				<geometry>
-					<mesh filename="package://QR/movo_description_drake/meshes/pan_tilt/collision/pan_tilt_base.obj" />
+					<mesh filename="package://QR/movo_description_drake/meshes/pan_tilt/visual/pan_tilt_base.obj" />
 				</geometry>
         <material>
@@ -77,5 +77,5 @@
 			<visual>
 				<geometry>
-					<mesh filename="package://QR/movo_description_drake/meshes/pan_tilt/collision/pan_link.obj" />
+					<mesh filename="package://QR/movo_description_drake/meshes/pan_tilt/visual/pan_link.obj" />
 				</geometry>
         <material>
@@ -116,5 +116,5 @@
 			<visual>
 				<geometry>
-					<mesh filename="package://QR/movo_description_drake/meshes/pan_tilt/collision/tilt_link.obj" />
+					<mesh filename="package://QR/movo_description_drake/meshes/pan_tilt/visual/tilt_link.obj" />
 				</geometry>
         <material>

File: movo_common/movo_description/urdf/sensors/kinect_one_sensor.urdf.xacro (robot description, xacro)
@@ -57,5 +57,5 @@
 			<visual>
 				<geometry>
-					<mesh filename="package://QR/movo_description_drake/meshes/sensors/collision/kinect_one_collision.obj" />
+					<mesh filename="package://QR/movo_description_drake/meshes/sensors/visual/kinect_one.obj" />
 				</geometry>
         <material>

File: movo_common/movo_description/urdf/sensors/sick_tim.urdf.xacro (robot description, xacro)
@@ -37,5 +37,5 @@
 <!--            <visual>
                 <geometry>
-                    <mesh filename="package://QR/movo_description_drake/meshes/sensors/collision/sick_tim.dae" />
+                    <mesh filename="package://QR/movo_description_drake/meshes/sensors/visual/sick_tim.dae" />
                 </geometry>
             </visual> -->

Commit message: fixup base collision geometry

File: movo_common/movo_description/urdf/movo_components/movo_base.urdf.xacro (robot description, xacro)
@@ -27,5 +27,5 @@
 SOFTWARE, EVEN IF ADVISED OF THE POSSIBILITY OF SUCH DAMAGE.
 -->
-<robot name="movo_base" xmlns:xacro="http://ros.org/wiki/xacro">
+<robot name="movo_base" xmlns:xacro="http://ros.org/wiki/xacro" xmlns:drake="http://drake.mit.edu">
     <xacro:include filename="$(find movo_description)/urdf/sensors/sick_tim.urdf.xacro" />
     <!-- Wheel Mounting Positions and Properties-->
@@ -89,5 +89,5 @@
         </gazebo>
         <joint name="base_chassis_joint" type="fixed">
-            <origin xyz="0 0 ${wheel_radius + 0.01}" rpy="0 0 0" />
+            <origin xyz="0 0 ${wheel_radius}" rpy="0 0 0" />
             <parent link="base_link" />
             <child link="base_chassis_link" />
@@ -101,4 +101,5 @@
                          izx="0" izy="0" izz="0.000714" />
 			</inertial>
+      <!-- russt: remove this to avoid collision with the ground and reduce unnecessary complexity.
             <collision>
 				<geometry>
@@ -106,4 +107,5 @@
 				</geometry>
 			</collision>
+      -->
 			<visual>
 				<origin xyz="0 0 0" rpy="0 0 0" />

File: movo_common/movo_description/urdf/movo_components/movo_body.urdf.xacro (robot description, xacro)
@@ -60,4 +60,11 @@
         </material>
 			</visual>
+      <!-- russt: add a box geometry surrounding the base -->
+      <collision>
+        <origin xyz="0 0 0.1071" />
+        <geometry>
+          <box size="0.8106 0.5097 0.3042" />
+        </geometry>
+      </collision>
 		</link>
         <joint name="upper_body_joint" type="fixed">
