Commit message: replace sammy's bogus inertias

File: movo_common/movo_description/urdf/manipulation/jaco/j2s7s300_arm_sphere_collision.urdf.xacro (robot description, xacro)
@@ -578,5 +578,5 @@
       <mass value="0.001"/>
       <origin xyz="0 0 -0.06"/>
-      <inertia ixx="0.001" ixy="0" ixz="0" iyy="0.001" iyz="0" izz="0.001"/>
+      <inertia ixx="0.000001" ixy="0" ixz="0" iyy="0.000001" iyz="0" izz="0.000001"/>
     </inertial>
   </link>

Commit message: working on robotiq model

File: movo_common/movo_description/urdf/manipulation/jaco/j2s7s300_arm_sphere_collision.urdf.xacro (robot description, xacro)
@@ -598,4 +598,10 @@
     </actuator>
   </transmission>
+    <joint name="${prefix}ee_fixed_joint" type="fixed">
+        <parent link="${prefix}link_7" />
+        <child link="${prefix}ee_link" />
+        <origin xyz="0 0 -0.1600" rpy="${M_PI} ${M_PI/2} 0"/>
+    </joint>
+    <link name="${prefix}ee_link"/>
   </xacro:macro>
 </robot>

File: movo_common/movo_description/urdf/manipulation/robotiq/robotiq_85_gripper.transmission.xacro (robot description, xacro)
@@ -2,4 +2,5 @@
 <robot xmlns:xacro="http://ros.org/wiki/xacro">
   <xacro:macro name="robotiq_85_gripper_transmission" params="prefix">
+        <!-- russt: i've fixed this joint
         <transmission name="${prefix}gripper_finger1_trans">
             <type>transmission_interface/SimpleTransmission</type>
@@ -12,4 +13,49 @@
             </actuator>
         </transmission>
+        -->
+        <!-- russt: add extra transmissions to overcome missing mimic joints -->
+        <!--
+        <transmission name="${prefix}gripper_finger1_inner_knuckle_trans">
+            <type>transmission_interface/SimpleTransmission</type>
+            <joint name="${prefix}gripper_finger1_inner_knuckle_joint">
+                <hardwareInterface>PositionJointInterface</hardwareInterface>
+            </joint>
+            <actuator name="${prefix}gripper_finger1_inner_knuckle_motor">
+                <mechanicalReduction>1</mechanicalReduction>
+                <hardwareInterface>PositionJointInterface</hardwareInterface>
+            </actuator>
+        </transmission>
+        <transmission name="${prefix}gripper_finger2_inner_knuckle_trans">
+            <type>transmission_interface/SimpleTransmission</type>
+            <joint name="${prefix}gripper_finger2_inner_knuckle_joint">
+                <hardwareInterface>PositionJointInterface</hardwareInterface>
+            </joint>
+            <actuator name="${prefix}gripper_finger2_inner_knuckle_motor">
+                <mechanicalReduction>1</mechanicalReduction>
+                <hardwareInterface>PositionJointInterface</hardwareInterface>
+            </actuator>
+        </transmission>
+        <transmission name="${prefix}gripper_finger1_finger_tip_trans">
+            <type>transmission_interface/SimpleTransmission</type>
+            <joint name="${prefix}gripper_finger1_finger_tip_joint">
+                <hardwareInterface>PositionJointInterface</hardwareInterface>
+            </joint>
+            <actuator name="${prefix}gripper_finger1_finger_tip_motor">
+                <mechanicalReduction>1</mechanicalReduction>
+                <hardwareInterface>PositionJointInterface</hardwareInterface>
+            </actuator>
+        </transmission>
+        <transmission name="${prefix}gripper_finger2_finger_tip_trans">
+            <type>transmission_interface/SimpleTransmission</type>
+            <joint name="${prefix}gripper_finger2_finger_tip_joint">
+                <hardwareInterface>PositionJointInterface</hardwareInterface>
+            </joint>
+            <actuator name="${prefix}gripper_finger2_finger_tip_motor">
+                <mechanicalReduction>1</mechanicalReduction>
+                <hardwareInterface>PositionJointInterface</hardwareInterface>
+            </actuator>
+        </transmission>
+        -->
+        <!-- russt: end new transmissions -->
         <gazebo>
                 <!-- loading plugin: mimic joints works in gazebo now -->

File: movo_common/movo_description/urdf/manipulation/robotiq/robotiq_85_gripper.urdf.xacro (robot description, xacro)
@@ -1,4 +1,4 @@
 <?xml version="1.0"?>
-<robot name="robotiq_85_gripper" xmlns:xacro="http://ros.org/wiki/xacro">
+<robot name="robotiq_85_gripper" xmlns:xacro="http://ros.org/wiki/xacro" xmlns:drake="http://drake.mit.edu">
     <xacro:include filename="$(find movo_description)/urdf/manipulation/robotiq/robotiq_85_gripper.transmission.xacro" />
     <xacro:property name="M_PI" value="3.14159"/>
@@ -66,5 +66,7 @@
             <kd>1.0</kd>
         </gazebo>
-        <joint name="${prefix}gripper_finger1_joint" type="revolute">
+        <!-- russt: fix this to overcome mimic
+        <joint name="${prefix}gripper_finger1_joint" type="revolute"> -->
+        <joint name="${prefix}gripper_finger1_joint" type="fixed">
             <parent link="${prefix}gripper_base_link"/>
             <child link="${prefix}gripper_finger1_knuckle_link"/>
@@ -73,5 +75,7 @@
             <limit lower="0.0" upper="0.804" velocity="2.0" effort="1000"/>
         </joint>
-        <joint name="${prefix}gripper_finger2_joint" type="revolute">
+        <!-- russt: fix this to overcome mimic
+        <joint name="${prefix}gripper_finger2_joint" type="revolute"> -->
+        <joint name="${prefix}gripper_finger2_joint" type="fixed">
             <parent link="${prefix}gripper_base_link"/>
             <child link="${prefix}gripper_finger2_knuckle_link"/>
@@ -79,5 +83,5 @@
             <origin rpy="0.0 0.0 0.0" xyz="0.05490451627 -0.03060114443 0.0"/>
             <limit lower="-3.14" upper="3.14" velocity="100.0" effort="1000"/>
-            <mimic joint="${prefix}gripper_finger1_joint"/>
+            <!-- russt: remove this until inverse dynamics supports it <mimic joint="${prefix}gripper_finger1_joint"/> -->
         </joint>
         <link name="${prefix}gripper_finger1_knuckle_link">
@@ -195,5 +199,7 @@
             <kd>1.0</kd>
         </gazebo>
-        <joint name="${prefix}gripper_finger1_inner_knuckle_joint" type="continuous">
+        <!-- russt: fix this for now
+        <joint name="${prefix}gripper_finger1_inner_knuckle_joint" type="continuous"> -->
+        <joint name="${prefix}gripper_finger1_inner_knuckle_joint" type="fixed">
             <parent link="${prefix}gripper_base_link"/>
             <child link="${prefix}gripper_finger1_inner_knuckle_link"/>
@@ -201,7 +207,11 @@
             <origin xyz="0.06142 0.0127 0" rpy="${M_PI} 0.0 0.0" />
             <limit lower="-3.14" upper="3.14" velocity="100.0" effort="0.1"/>
+            <!-- russt: remove this for now
             <mimic joint="${prefix}gripper_finger1_joint" offset="0"/>
-        </joint>
-        <joint name="${prefix}gripper_finger2_inner_knuckle_joint" type="continuous">
+            -->
+        </joint>
+        <!-- russt: fix this for now
+        <joint name="${prefix}gripper_finger2_inner_knuckle_joint" type="continuous"> -->
+        <joint name="${prefix}gripper_finger2_inner_knuckle_joint" type="fixed">
             <parent link="${prefix}gripper_base_link"/>
             <child link="${prefix}gripper_finger2_inner_knuckle_link"/>
@@ -209,5 +219,7 @@
             <origin xyz="0.06142 -0.0127 0" rpy="0 0 0"/>
             <limit lower="-3.14" upper="3.14" velocity="100.0" effort="0.1"/>
+            <!-- russt: remove this for now
             <mimic joint="${prefix}gripper_finger1_joint" offset="0"/>
+            -->
         </joint>
         <link name="${prefix}gripper_finger1_inner_knuckle_link">
@@ -263,5 +275,7 @@
             <kd>1.0</kd>
         </gazebo>
-        <joint name="${prefix}gripper_finger1_finger_tip_joint" type="continuous">
+        <!-- russt: fix this for now
+        <joint name="${prefix}gripper_finger1_finger_tip_joint" type="continuous">-->
+        <joint name="${prefix}gripper_finger1_finger_tip_joint" type="fixed">
             <parent link="${prefix}gripper_finger1_inner_knuckle_link"/>
             <child link="${prefix}gripper_finger1_finger_tip_link"/>
@@ -269,7 +283,11 @@
             <origin xyz="0.04303959807 -0.03759940821 0.0" rpy="0.0 0.0 0.0"/>
             <limit lower="-3.14" upper="3.14" velocity="100.0" effort="0.1"/>
+            <!-- russt: remove this for now
             <mimic joint="${prefix}gripper_finger1_joint" multiplier="-1"/>
-        </joint>
-        <joint name="${prefix}gripper_finger2_finger_tip_joint" type="continuous">
+            -->
+        </joint>
+        <!-- russt: fix this for now
+        <joint name="${prefix}gripper_finger2_finger_tip_joint" type="continuous"> -->
+        <joint name="${prefix}gripper_finger2_finger_tip_joint" type="fixed">
             <parent link="${prefix}gripper_finger2_inner_knuckle_link"/>
             <child link="${prefix}gripper_finger2_finger_tip_link"/>
@@ -277,5 +295,7 @@
             <origin rpy="0.0 0.0 0.0" xyz="0.04303959807 -0.03759940821  0.0"/>
             <limit lower="-3.14" upper="3.14" velocity="100.0" effort="0.1"/>
+            <!-- russt: remove this for now
             <mimic joint="${prefix}gripper_finger1_joint" multiplier="-1"/>
+            -->
         </joint>
         <link name="${prefix}gripper_finger1_finger_tip_link">
@@ -332,4 +352,24 @@
         </gazebo>
         <xacro:robotiq_85_gripper_transmission prefix="${prefix}" />
+        <drake:collision_filter_group name="${prefix}link_6_coupler">
+          <drake:member link="${prefix}link_6" />
+          <drake:member link="${prefix}robotiq_coupler_link" />
+          <drake:member link="${prefix}gripper_base_link" />
+          <drake:ignored_collision_filter_group name="${prefix}link_6_coupler" />
+        </drake:collision_filter_group>
+        <drake:collision_filter_group name="${prefix}finger_1">
+          <drake:member link="${prefix}gripper_finger1_finger_link" />
+          <drake:member link="${prefix}gripper_finger1_inner_knuckle_link" />
+          <drake:member link="${prefix}gripper_finger1_knuckle_link" />
+          <drake:member link="${prefix}gripper_finger1_finger_tip_link" />
+          <drake:ignored_collision_filter_group name="${prefix}finger_1" />
+        </drake:collision_filter_group>
+        <drake:collision_filter_group name="${prefix}finger_2">
+          <drake:member link="${prefix}gripper_finger2_finger_link" />
+          <drake:member link="${prefix}gripper_finger2_inner_knuckle_link" />
+          <drake:member link="${prefix}gripper_finger2_knuckle_link" />
+          <drake:member link="${prefix}gripper_finger2_finger_tip_link" />
+          <drake:ignored_collision_filter_group name="${prefix}finger_2" />
+        </drake:collision_filter_group>
     </xacro:macro>
 </robot>
