Commit message: make j2s7 files match joint names and joint zeros in jaco_7dof

File: movo_common/movo_description/urdf/manipulation/jaco/j2s7s300_arm_sphere_collision.urdf.xacro (robot description, xacro)
@@ -118,5 +118,5 @@
     </inertial>
   </link>
-  <joint name="${prefix}joint_1" type="continuous">
+  <joint name="${prefix}shoulder_pan_joint" type="continuous">
     <parent link="${prefix}link_base"/>
     <child link="${prefix}link_1"/>
@@ -132,5 +132,5 @@
   <transmission name="${prefix}joint_1_trans">
     <type>transmission_interface/SimpleTransmission</type>
-    <joint name="${prefix}joint_1">
+    <joint name="${prefix}shoulder_pan_joint">
       <hardwareInterface>EffortJointInterface</hardwareInterface>
     </joint>
@@ -222,15 +222,15 @@
     </inertial>
   </link>
-  <joint name="${prefix}joint_2" type="revolute">
+  <joint name="${prefix}shoulder_lift_joint" type="revolute">
     <parent link="${prefix}link_1"/>
     <child link="${prefix}link_2"/>
     <axis xyz="0 0 1"/>
-    <limit effort="2000" lower="0.523598775598" upper="5.75958653158" velocity="0.63"/>
-    <origin rpy="-1.57079632679 0 3.14159265359" xyz="0 0.0016 -0.11875"/>
+    <limit effort="2000" lower="${0.523598775598 - M_PI}" upper="${5.75958653158 - M_PI}" velocity="0.63"/>
+    <origin rpy="1.57079632679 0 0" xyz="0 0.0016 -0.11875"/>
     <dynamics damping="0.01" friction="0.0"/>
   </joint>
   <transmission name="${prefix}joint_2_trans">
     <type>transmission_interface/SimpleTransmission</type>
-    <joint name="${prefix}joint_2">
+    <joint name="${prefix}shoulder_lift_joint">
       <hardwareInterface>EffortJointInterface</hardwareInterface>
     </joint>
@@ -328,5 +328,5 @@
     </inertial>
   </link>
-  <joint name="${prefix}joint_3" type="continuous">
+  <joint name="${prefix}arm_half_joint" type="continuous">
     <parent link="${prefix}link_2"/>
     <child link="${prefix}link_3"/>
@@ -338,5 +338,5 @@
   <transmission name="${prefix}joint_3_trans">
     <type>transmission_interface/SimpleTransmission</type>
-    <joint name="${prefix}joint_3">
+    <joint name="${prefix}arm_half_joint">
       <hardwareInterface>EffortJointInterface</hardwareInterface>
     </joint>
@@ -440,15 +440,15 @@
     </inertial>
   </link>
-  <joint name="${prefix}joint_4" type="revolute">
+  <joint name="${prefix}elbow_joint" type="revolute">
     <parent link="${prefix}link_3"/>
     <child link="${prefix}link_4"/>
     <axis xyz="0 0 1"/>
-    <limit effort="2000" lower="0.523598775598" upper="5.75958653158" velocity="0.63"/>
-    <origin rpy="1.57079632679 0 3.14159265359" xyz="0 0 -0.205"/>
+    <limit effort="2000" lower="${0.523598775598 - M_PI}" upper="${5.75958653158 - M_PI}" velocity="0.63"/>
+    <origin rpy="-1.57079632679 0 0" xyz="0 0 -0.205"/>
     <dynamics damping="0.01" friction="0.0"/>
   </joint>
   <transmission name="${prefix}joint_4_trans">
     <type>transmission_interface/SimpleTransmission</type>
-    <joint name="${prefix}joint_4">
+    <joint name="${prefix}elbow_joint">
       <hardwareInterface>EffortJointInterface</hardwareInterface>
     </joint>
@@ -498,5 +498,5 @@
     </inertial>
   </link>
-  <joint name="${prefix}joint_5" type="continuous">
+  <joint name="${prefix}wrist_spherical_1_joint" type="continuous">
     <parent link="${prefix}link_4"/>
     <child link="${prefix}link_5"/>
@@ -508,5 +508,5 @@
   <transmission name="${prefix}joint_5_trans">
     <type>transmission_interface/SimpleTransmission</type>
-    <joint name="${prefix}joint_5">
+    <joint name="${prefix}wrist_spherical_1_joint">
       <hardwareInterface>EffortJointInterface</hardwareInterface>
     </joint>
@@ -550,15 +550,15 @@
     </inertial>
   </link>
-  <joint name="${prefix}joint_6" type="revolute">
+  <joint name="${prefix}wrist_spherical_2_joint" type="revolute">
     <parent link="${prefix}link_5"/>
     <child link="${prefix}link_6"/>
     <axis xyz="0 0 1"/>
-    <limit effort="2000" lower="0.523598775598" upper="5.75958653158" velocity="0.85"/>
-    <origin rpy="1.57079632679 0 3.14159265359" xyz="0 0 -0.10375"/>
+    <limit effort="2000" lower="${0.523598775598 - M_PI}" upper="${5.75958653158 - M_PI}" velocity="0.85"/>
+    <origin rpy="-1.57079632679 0 0" xyz="0 0 -0.10375"/>
     <dynamics damping="0.01" friction="0.0"/>
   </joint>
   <transmission name="${prefix}joint_6_trans">
     <type>transmission_interface/SimpleTransmission</type>
-    <joint name="${prefix}joint_6">
+    <joint name="${prefix}wrist_spherical_2_joint">
       <hardwareInterface>EffortJointInterface</hardwareInterface>
     </joint>
@@ -581,5 +581,5 @@
     </inertial>
   </link>
-  <joint name="${prefix}joint_7" type="continuous">
+  <joint name="${prefix}wrist_3_joint" type="continuous">
     <parent link="${prefix}link_6"/>
     <child link="${prefix}link_7"/>
@@ -591,5 +591,5 @@
   <transmission name="${prefix}joint_7_trans">
     <type>transmission_interface/SimpleTransmission</type>
-    <joint name="${prefix}joint_7">
+    <joint name="${prefix}wrist_3_joint">
       <hardwareInterface>EffortJointInterface</hardwareInterface>
     </joint>

File: movo_common/movo_description/urdf/manipulation/jaco/jaco.urdf.xacro (robot description, xacro)
@@ -47,5 +47,5 @@
             <visual>
                 <geometry>
-                <mesh filename="package://QR/movo_description_drake/meshes/manipulation/jaco/visual/base.dae"/>
+                <mesh filename="package://QR/movo_description_drake/meshes/manipulation/jaco/visual/base.obj"/>
                 </geometry>
             </visual>
@@ -83,5 +83,5 @@
             <visual>
                 <geometry>
-                    <mesh filename="package://QR/movo_description_drake/meshes/manipulation/jaco/visual/shoulder.dae"/>
+                    <mesh filename="package://QR/movo_description_drake/meshes/manipulation/jaco/visual/shoulder.obj"/>
                 </geometry>
             </visual>
@@ -119,5 +119,5 @@
             <visual>
                 <geometry>
-                    <mesh filename="package://QR/movo_description_drake/meshes/manipulation/jaco/visual/upper_arm.dae"/>
+                    <mesh filename="package://QR/movo_description_drake/meshes/manipulation/jaco/visual/upper_arm.obj"/>
                 </geometry>
             </visual>
@@ -155,5 +155,5 @@
             <visual>
                 <geometry>
-                    <mesh filename="package://QR/movo_description_drake/meshes/manipulation/jaco/visual/forearm.dae"/>
+                    <mesh filename="package://QR/movo_description_drake/meshes/manipulation/jaco/visual/forearm.obj"/>
                 </geometry>
             </visual>
@@ -182,5 +182,5 @@
             <visual>
                 <geometry>
-                    <mesh filename="package://QR/movo_description_drake/meshes/manipulation/jaco/visual/wrist_1.dae"/>
+                    <mesh filename="package://QR/movo_description_drake/meshes/manipulation/jaco/visual/wrist_1.obj"/>
                 </geometry>
             </visual>
@@ -218,5 +218,5 @@
             <visual>
                 <geometry>
-                    <mesh filename="package://QR/movo_description_drake/meshes/manipulation/jaco/visual/wrist_2.dae"/>
+                    <mesh filename="package://QR/movo_description_drake/meshes/manipulation/jaco/visual/wrist_2.obj"/>
                 </geometry>
             </visual>
@@ -254,5 +254,5 @@
             <visual>
                 <geometry>
-                    <mesh filename="package://QR/movo_description_drake/meshes/manipulation/jaco/visual/kinova_actuator_gearing.dae"/>
+                    <mesh filename="package://QR/movo_description_drake/meshes/manipulation/jaco/visual/kinova_actuator_gearing.obj"/>
                 </geometry>
             </visual>

File: movo_common/movo_description/urdf/manipulation/jaco/jaco_7dof.urdf.xacro (robot description, xacro)
@@ -55,5 +55,5 @@
             <visual>
                 <geometry>
-                <mesh filename="package://QR/movo_description_drake/meshes/manipulation/jaco/visual/base.dae"/>
+                <mesh filename="package://QR/movo_description_drake/meshes/manipulation/jaco/visual/base.obj"/>
                 </geometry>
             </visual>
@@ -91,5 +91,5 @@
             <visual>
                 <geometry>
-                    <mesh filename="package://QR/movo_description_drake/meshes/manipulation/jaco/visual/shoulder_7dof.dae"/>
+                    <mesh filename="package://QR/movo_description_drake/meshes/manipulation/jaco/visual/shoulder_7dof.obj"/>
                 </geometry>
             </visual>
@@ -127,5 +127,5 @@
             <visual>
                 <geometry>
-                    <mesh filename="package://QR/movo_description_drake/meshes/manipulation/jaco/visual/arm_half_1.dae"/>
+                    <mesh filename="package://QR/movo_description_drake/meshes/manipulation/jaco/visual/arm_half_1.obj"/>
                 </geometry>
             </visual>
@@ -163,5 +163,5 @@
             <visual>
                 <geometry>
-                    <mesh filename="package://QR/movo_description_drake/meshes/manipulation/jaco/visual/arm_half_2.dae"/>
+                    <mesh filename="package://QR/movo_description_drake/meshes/manipulation/jaco/visual/arm_half_2.obj"/>
                 </geometry>
             </visual>
@@ -199,5 +199,5 @@
             <visual>
                 <geometry>
-                    <mesh filename="package://QR/movo_description_drake/meshes/manipulation/jaco/visual/forearm_7dof.dae"/>
+                    <mesh filename="package://QR/movo_description_drake/meshes/manipulation/jaco/visual/forearm_7dof.obj"/>
                 </geometry>
             </visual>
@@ -227,5 +227,5 @@
             <visual>
                 <geometry>
-                    <mesh filename="package://QR/movo_description_drake/meshes/manipulation/jaco/visual/wrist_spherical_1.dae"/>
+                    <mesh filename="package://QR/movo_description_drake/meshes/manipulation/jaco/visual/wrist_spherical_1.obj"/>
                 </geometry>
             </visual>
@@ -263,5 +263,5 @@
             <visual>
                 <geometry>
-                    <mesh filename="package://QR/movo_description_drake/meshes/manipulation/jaco/visual/wrist_spherical_2.dae"/>
+                    <mesh filename="package://QR/movo_description_drake/meshes/manipulation/jaco/visual/wrist_spherical_2.obj"/>
                 </geometry>
             </visual>
@@ -299,5 +299,5 @@
             <visual>
                 <geometry>
-                    <mesh filename="package://QR/movo_description_drake/meshes/manipulation/jaco/visual/kinova_actuator_gearing.dae"/>
+                    <mesh filename="package://QR/movo_description_drake/meshes/manipulation/jaco/visual/kinova_actuator_gearing.obj"/>
                 </geometry>
             </visual>

File: movo_common/movo_description/urdf/manipulation/robotiq/robotiq_85_gripper.urdf.xacro (robot description, xacro)
@@ -10,5 +10,5 @@
     </xacro:unless>
     <xacro:if value="$(optenv WELD_FINGERS false)">
-      <xacro:property name="revolute_or_fixed" value="${revolute_or_fixed_1}"/>
+      <xacro:property name="revolute_or_fixed" value="fixed"/>
     </xacro:if>
     <xacro:unless value="$(optenv WELD_FINGERS false)">

File: movo_common/movo_description/urdf/movo.urdf.xacro (robot description, xacro)
@@ -35,5 +35,5 @@
     <!-- russt: use modified drake version for now
     <xacro:include filename="$(find movo_description)/urdf/manipulation/kinova_grippers/kg3_gripper.urdf.xacro" /> -->
-    <xacro:include filename="$(find movo_description)/urdf/manipulation/kinova_grippers/j2s7s300_hand_sphere_collision.urdf.xacro" /> -->
+    <xacro:include filename="$(find movo_description)/urdf/manipulation/kinova_grippers/j2s7s300_hand_sphere_collision.urdf.xacro" />
     <xacro:include filename="$(find movo_description)/urdf/manipulation/kinova_grippers/kg2_gripper.urdf.xacro" />
     <xacro:include filename="$(find movo_description)/urdf/gzplugin_grasp_fix.urdf.xacro" />

File: movo_common/movo_description/urdf/sensors/sick_tim.urdf.xacro (robot description, xacro)
@@ -37,5 +37,5 @@
 <!--            <visual>
                 <geometry>
-                    <mesh filename="package://QR/movo_description_drake/meshes/sensors/visual/sick_tim.dae" />
+                    <mesh filename="package://QR/movo_description_drake/meshes/sensors/visual/sick_tim.obj" />
                 </geometry>
             </visual> -->
