Commit message: fix sdf inertias and add material names

File: movo_common/movo_description/urdf/manipulation/jaco/j2s7s300_arm_sphere_collision.urdf.xacro (robot description, xacro)
@@ -13,5 +13,5 @@
         <mesh filename="package://drake_models/jaco_description/meshes/base.obj"/>
       </geometry>
-      <material>
+      <material name="black">
         <color rgba="0.1788232 0.1788232 0.1788232 1"/>
       </material>
@@ -58,5 +58,5 @@
         <mesh filename="package://drake_models/jaco_description/meshes/shoulder.obj"/>
       </geometry>
-      <material>
+      <material name="black">
         <color rgba="0.1788232 0.1788232 0.1788232 1"/>
       </material>
@@ -66,5 +66,5 @@
         <mesh filename="package://drake_models/jaco_description/meshes/ring_big.obj"/>
       </geometry>
-      <material>
+      <material name="black">
         <color rgba="0.627451 0.627451 0.627451 1"/>
       </material>
@@ -144,5 +144,5 @@
         <mesh filename="package://drake_models/jaco_description/meshes/arm_half_1.obj"/>
       </geometry>
-      <material>
+      <material name="black">
         <color rgba="0.1788232 0.1788232 0.1788232 1"/>
       </material>
@@ -152,5 +152,5 @@
         <mesh filename="package://drake_models/jaco_description/meshes/ring_big.obj"/>
       </geometry>
-      <material>
+      <material name="black">
         <color rgba="0.627451 0.627451 0.627451 1"/>
       </material>
@@ -244,5 +244,5 @@
         <mesh filename="package://drake_models/jaco_description/meshes/arm_half_2.obj"/>
       </geometry>
-      <material>
+      <material name="black">
         <color rgba="0.1788232 0.1788232 0.1788232 1"/>
       </material>
@@ -252,5 +252,5 @@
         <mesh filename="package://drake_models/jaco_description/meshes/ring_big.obj"/>
       </geometry>
-      <material>
+      <material name="black">
         <color rgba="0.627451 0.627451 0.627451 1"/>
       </material>
@@ -350,5 +350,5 @@
         <mesh filename="package://drake_models/jaco_description/meshes/forearm.obj"/>
       </geometry>
-      <material>
+      <material name="black">
         <color rgba="0.1788232 0.1788232 0.1788232 1"/>
       </material>
@@ -358,5 +358,5 @@
         <mesh filename="package://drake_models/jaco_description/meshes/ring_small.obj"/>
       </geometry>
-      <material>
+      <material name="black">
         <color rgba="0.627451 0.627451 0.627451 1"/>
       </material>
@@ -462,5 +462,5 @@
         <mesh filename="package://drake_models/jaco_description/meshes/wrist_spherical_1.obj"/>
       </geometry>
-      <material>
+      <material name="black">
         <color rgba="0.1788232 0.1788232 0.1788232 1"/>
       </material>
@@ -470,5 +470,5 @@
         <mesh filename="package://drake_models/jaco_description/meshes/ring_small.obj"/>
       </geometry>
-      <material>
+      <material name="black">
         <color rgba="0.627451 0.627451 0.627451 1"/>
       </material>
@@ -520,5 +520,5 @@
         <mesh filename="package://drake_models/jaco_description/meshes/wrist_spherical_2.obj"/>
       </geometry>
-      <material>
+      <material name="black">
         <color rgba="0.1788232 0.1788232 0.1788232 1"/>
       </material>
@@ -528,5 +528,5 @@
         <mesh filename="package://drake_models/jaco_description/meshes/ring_small.obj"/>
       </geometry>
-      <material>
+      <material name="black">
         <color rgba="0.627451 0.627451 0.627451 1"/>
       </material>

File: movo_common/movo_description/urdf/manipulation/kinova_grippers/j2s7s300_hand_sphere_collision.urdf.xacro (robot description, xacro)
@@ -17,5 +17,5 @@
         <mesh filename="package://drake_models/jaco_description/meshes/hand_3finger.obj"/>
       </geometry>
-      <material>
+      <material name="black">
         <color rgba="0.1788232 0.1788232 0.1788232 1"/>
       </material>
@@ -25,5 +25,5 @@
         <mesh filename="package://drake_models/jaco_description/meshes/ring_small.obj"/>
       </geometry>
-      <material>
+      <material name="black">
         <color rgba="0.627451 0.627451 0.627451 1"/>
       </material>
@@ -107,5 +107,5 @@
         <mesh filename="package://drake_models/jaco_description/meshes/finger_proximal.obj"/>
       </geometry>
-      <material>
+      <material name="black">
         <color rgba="0.5960783 0.5960783 0.5960783 1"/>
       </material>
@@ -163,5 +163,5 @@
         <mesh filename="package://drake_models/jaco_description/meshes/finger_distal.obj"/>
       </geometry>
-      <material>
+      <material name="black">
         <color rgba="0.5960783 0.5960783 0.5960783 1"/>
       </material>
@@ -215,5 +215,5 @@
         <mesh filename="package://drake_models/jaco_description/meshes/finger_proximal.obj"/>
       </geometry>
-      <material>
+      <material name="black">
         <color rgba="0.5960783 0.5960783 0.5960783 1"/>
       </material>
@@ -271,5 +271,5 @@
         <mesh filename="package://drake_models/jaco_description/meshes/finger_distal.obj"/>
       </geometry>
-      <material>
+      <material name="black">
         <color rgba="0.5960783 0.5960783 0.5960783 1"/>
       </material>
@@ -323,5 +323,5 @@
         <mesh filename="package://drake_models/jaco_description/meshes/finger_proximal.obj"/>
       </geometry>
-      <material>
+      <material name="black">
         <color rgba="0.5960783 0.5960783 0.5960783 1"/>
       </material>
@@ -379,5 +379,5 @@
         <mesh filename="package://drake_models/jaco_description/meshes/finger_distal.obj"/>
       </geometry>
-      <material>
+      <material name="black">
         <color rgba="0.5960783 0.5960783 0.5960783 1"/>
       </material>

File: movo_common/movo_description/urdf/manipulation/kinova_grippers/kg2_gripper.urdf.xacro (robot description, xacro)
@@ -57,15 +57,9 @@
             </collision>
             <inertial>
-                <!-- russt: replace these using drake's mesh_to_sdf -->
-                <pose>0.000925589 -0.0179473 4.08395e-09 0 0 0</pose>
-                <mass>0.006837878460055832</mass>
-                <inertia>
-                  <ixx>1.2773e-06</ixx>
-                  <ixy>7.66328e-08</ixy>
-                  <ixz>-1.1905e-13</ixz>
-                  <iyy>2.50863e-07</iyy>
-                  <iyz>4.97761e-13</iyz>
-                  <izz>1.38456e-06</izz>
-                </inertia>
+                <!-- russt: replaced these using drake's mesh_to_sdf -->
+                <origin xyz="0.000925589 -0.0179473 4.08395e-09"/>
+                <mass value="0.006837878460055832" />
+                <inertia ixx="1.2773e-06"  ixy="7.66328e-08" ixz="-1.1905e-13"
+                         iyy="2.50863e-07" iyz="4.97761e-13" izz="1.38456e-06"/>
                 <!-- these original values aren't physically valid
                 <mass value="0.009127" />
@@ -105,15 +99,9 @@
             </collision>
             <inertial>
-                <!-- russt: replace these using drake's mesh_to_sdf -->
-                <pose>0.000925589 -0.0179473 4.08395e-09 0 0 0</pose>
-                <mass>0.006837878460055832</mass>
-                <inertia>
-                  <ixx>1.2773e-06</ixx>
-                  <ixy>7.66328e-08</ixy>
-                  <ixz>-1.1905e-13</ixz>
-                  <iyy>2.50863e-07</iyy>
-                  <iyz>4.97761e-13</iyz>
-                  <izz>1.38456e-06</izz>
-                </inertia>
+                <!-- russt: replaced these using drake's mesh_to_sdf -->
+                <origin xyz="0.000925589 -0.0179473 4.08395e-09"/>
+                <mass value="0.006837878460055832" />
+                <inertia ixx="1.2773e-06"  ixy="7.66328e-08" ixz="-1.1905e-13"
+                         iyy="2.50863e-07" iyz="4.97761e-13" izz="1.38456e-06"/>
                 <!-- these original values aren't physically valid
                 <mass value="0.009127" />
@@ -152,14 +140,8 @@
             <inertial>
                 <!-- russt: set these using drake's mesh to sdf -->
-                <pose>0.0148543 -0.00150728 -1.56703e-09 0 0 0</pose>
-                <mass>0.012779909194886162</mass>
-                <inertia>
-                  <ixx>1.05756e-06</ixx>
-                  <ixy>-9.59984e-07</ixy>
-                  <ixz>2.26386e-13</ixz>
-                  <iyy>3.44081e-06</iyy>
-                  <iyz>-1.09241e-14</iyz>
-                  <izz>3.8057e-06</izz>
-                </inertia>
+                <origin xyz="0.0148543 -0.00150728 -1.56703e-09" />
+                <mass value="0.012779909194886162" />
+                <inertia ixx="1.05756e-06" ixy="-9.59984e-07" ixz="2.26386e-13"
+                         iyy="3.44081e-06" iyz="-1.09241e-14" izz="3.8057e-06" />
                 <!-- these original values aren't physically valid
                 <mass value="0.012690" />
@@ -198,14 +180,8 @@
             <inertial>
                 <!-- russt: set these using drake's mesh to sdf -->
-                <pose>0.0148543 -0.00150728 -1.56703e-09 0 0 0</pose>
-                <mass>0.012779909194886162</mass>
-                <inertia>
-                  <ixx>1.05756e-06</ixx>
-                  <ixy>-9.59984e-07</ixy>
-                  <ixz>2.26386e-13</ixz>
-                  <iyy>3.44081e-06</iyy>
-                  <iyz>-1.09241e-14</iyz>
-                  <izz>3.8057e-06</izz>
-                </inertia>
+                <origin xyz="0.0148543 -0.00150728 -1.56703e-09" />
+                <mass value="0.012779909194886162" />
+                <inertia ixx="1.05756e-06" ixy="-9.59984e-07" ixz="2.26386e-13"
+                         iyy="3.44081e-06" iyz="-1.09241e-14" izz="3.8057e-06" />
                 <!-- these original values aren't physically valid
                 <mass value="0.012690" />

File: movo_common/movo_description/urdf/manipulation/kinova_grippers/kg3_gripper.urdf.xacro (robot description, xacro)
@@ -56,15 +56,9 @@
             </collision>
             <inertial>
-                <!-- russt: replace these using drake's mesh_to_sdf -->
-                <pose>0.000925589 -0.0179473 4.08395e-09 0 0 0</pose>
-                <mass>0.006837878460055832</mass>
-                <inertia>
-                  <ixx>1.2773e-06</ixx>
-                  <ixy>7.66328e-08</ixy>
-                  <ixz>-1.1905e-13</ixz>
-                  <iyy>2.50863e-07</iyy>
-                  <iyz>4.97761e-13</iyz>
-                  <izz>1.38456e-06</izz>
-                </inertia>
+                <!-- russt: replaced these using drake's mesh_to_sdf -->
+                <origin xyz="0.000925589 -0.0179473 4.08395e-09"/>
+                <mass value="0.006837878460055832" />
+                <inertia ixx="1.2773e-06"  ixy="7.66328e-08" ixz="-1.1905e-13"
+                         iyy="2.50863e-07" iyz="4.97761e-13" izz="1.38456e-06"/>
                 <!-- these original values aren't physically valid
                 <mass value="0.009127" />
@@ -105,15 +99,9 @@
             </collision>
             <inertial>
-                <!-- russt: replace these using drake's mesh_to_sdf -->
-                <pose>0.000925589 -0.0179473 4.08395e-09 0 0 0</pose>
-                <mass>0.006837878460055832</mass>
-                <inertia>
-                  <ixx>1.2773e-06</ixx>
-                  <ixy>7.66328e-08</ixy>
-                  <ixz>-1.1905e-13</ixz>
-                  <iyy>2.50863e-07</iyy>
-                  <iyz>4.97761e-13</iyz>
-                  <izz>1.38456e-06</izz>
-                </inertia>
+                <!-- russt: replaced these using drake's mesh_to_sdf -->
+                <origin xyz="0.000925589 -0.0179473 4.08395e-09"/>
+                <mass value="0.006837878460055832" />
+                <inertia ixx="1.2773e-06"  ixy="7.66328e-08" ixz="-1.1905e-13"
+                         iyy="2.50863e-07" iyz="4.97761e-13" izz="1.38456e-06"/>
                 <!-- these original values aren't physically valid
                 <mass value="0.009127" />
@@ -154,15 +142,9 @@
             </collision>
             <inertial>
-                <!-- russt: replace these using drake's mesh_to_sdf -->
-                <pose>0.000925589 -0.0179473 4.08395e-09 0 0 0</pose>
-                <mass>0.006837878460055832</mass>
-                <inertia>
-                  <ixx>1.2773e-06</ixx>
-                  <ixy>7.66328e-08</ixy>
-                  <ixz>-1.1905e-13</ixz>
-                  <iyy>2.50863e-07</iyy>
-                  <iyz>4.97761e-13</iyz>
-                  <izz>1.38456e-06</izz>
-                </inertia>
+                <!-- russt: replaced these using drake's mesh_to_sdf -->
+                <origin xyz="0.000925589 -0.0179473 4.08395e-09"/>
+                <mass value="0.006837878460055832" />
+                <inertia ixx="1.2773e-06"  ixy="7.66328e-08" ixz="-1.1905e-13"
+                         iyy="2.50863e-07" iyz="4.97761e-13" izz="1.38456e-06"/>
                 <!-- these original values aren't physically valid
                 <mass value="0.009127" />
@@ -201,14 +183,8 @@
             <inertial>
                 <!-- russt: set these using drake's mesh to sdf -->
-                <pose>0.0148543 -0.00150728 -1.56703e-09 0 0 0</pose>
-                <mass>0.012779909194886162</mass>
-                <inertia>
-                  <ixx>1.05756e-06</ixx>
-                  <ixy>-9.59984e-07</ixy>
-                  <ixz>2.26386e-13</ixz>
-                  <iyy>3.44081e-06</iyy>
-                  <iyz>-1.09241e-14</iyz>
-                  <izz>3.8057e-06</izz>
-                </inertia>
+                <origin xyz="0.0148543 -0.00150728 -1.56703e-09" />
+                <mass value="0.012779909194886162" />
+                <inertia ixx="1.05756e-06" ixy="-9.59984e-07" ixz="2.26386e-13"
+                         iyy="3.44081e-06" iyz="-1.09241e-14" izz="3.8057e-06" />
                 <!-- these original values aren't physically valid
                 <mass value="0.012690" />
@@ -247,14 +223,8 @@
             <inertial>
                 <!-- russt: set these using drake's mesh to sdf -->
-                <pose>0.0148543 -0.00150728 -1.56703e-09 0 0 0</pose>
-                <mass>0.012779909194886162</mass>
-                <inertia>
-                  <ixx>1.05756e-06</ixx>
-                  <ixy>-9.59984e-07</ixy>
-                  <ixz>2.26386e-13</ixz>
-                  <iyy>3.44081e-06</iyy>
-                  <iyz>-1.09241e-14</iyz>
-                  <izz>3.8057e-06</izz>
-                </inertia>
+                <origin xyz="0.0148543 -0.00150728 -1.56703e-09" />
+                <mass value="0.012779909194886162" />
+                <inertia ixx="1.05756e-06" ixy="-9.59984e-07" ixz="2.26386e-13"
+                         iyy="3.44081e-06" iyz="-1.09241e-14" izz="3.8057e-06" />
                 <!-- these original values aren't physically valid
                 <mass value="0.012690" />
@@ -293,14 +263,8 @@
             <inertial>
                 <!-- russt: set these using drake's mesh to sdf -->
-                <pose>0.0148543 -0.00150728 -1.56703e-09 0 0 0</pose>
-                <mass>0.012779909194886162</mass>
-                <inertia>
-                  <ixx>1.05756e-06</ixx>
-                  <ixy>-9.59984e-07</ixy>
-                  <ixz>2.26386e-13</ixz>
-                  <iyy>3.44081e-06</iyy>
-                  <iyz>-1.09241e-14</iyz>
-                  <izz>3.8057e-06</izz>
-                </inertia>
+                <origin xyz="0.0148543 -0.00150728 -1.56703e-09" />
+                <mass value="0.012779909194886162" />
+                <inertia ixx="1.05756e-06" ixy="-9.59984e-07" ixz="2.26386e-13"
+                         iyy="3.44081e-06" iyz="-1.09241e-14" izz="3.8057e-06" />
                 <!-- these original values aren't physically valid
                 <mass value="0.012690" />

File: movo_common/movo_description/urdf/movo_components/movo_base.urdf.xacro (robot description, xacro)
@@ -110,5 +110,5 @@
 					<mesh filename="package://QR/movo_description_drake/meshes/movo_components/visual/vector_base.obj" />
 				</geometry>
-        <material>
+        <material name="black">
           <color rgba="0.1788232 0.1788232 0.1788232 1"/>
         </material>

File: movo_common/movo_description/urdf/movo_components/movo_body.urdf.xacro (robot description, xacro)
@@ -56,5 +56,5 @@
 					<mesh filename="package://QR/movo_description_drake/meshes/movo_body/movo_lower_body.obj" />
 				</geometry>
-        <material>
+        <material name="black">
           <color rgba="0.1788232 0.1788232 0.1788232 1"/>
         </material>
@@ -79,5 +79,5 @@
 					<mesh filename="package://QR/movo_description_drake/meshes/movo_body/movo_upper_body.obj" />
 				</geometry>
-        <material>
+        <material name="black">
           <color rgba="0.1788232 0.1788232 0.1788232 1"/>
         </material>
@@ -118,5 +118,5 @@
 					<mesh filename="package://QR/movo_description_drake/meshes/movo_body/movo_mid_body.obj" />
 				</geometry>
-        <material>
+        <material name="black">
           <color rgba="0.1788232 0.1788232 0.1788232 1"/>
         </material>

File: movo_common/movo_description/urdf/movo_components/movo_pan_tilt.urdf.xacro (robot description, xacro)
@@ -41,5 +41,5 @@
 					<mesh filename="package://QR/movo_description_drake/meshes/pan_tilt/visual/pan_tilt_base.obj" />
 				</geometry>
-        <material>
+        <material name="black">
           <color rgba="0.1788232 0.1788232 0.1788232 1"/>
         </material>
@@ -79,5 +79,5 @@
 					<mesh filename="package://QR/movo_description_drake/meshes/pan_tilt/visual/pan_link.obj" />
 				</geometry>
-        <material>
+        <material name="black">
           <color rgba="0.1788232 0.1788232 0.1788232 1"/>
         </material>
@@ -118,5 +118,5 @@
 					<mesh filename="package://QR/movo_description_drake/meshes/pan_tilt/visual/tilt_link.obj" />
 				</geometry>
-        <material>
+        <material name="black">
           <color rgba="0.1788232 0.1788232 0.1788232 1"/>
         </material>

File: movo_common/movo_description/urdf/sensors/kinect_one_sensor.urdf.xacro (robot description, xacro)
@@ -37,14 +37,8 @@
             <inertial>
                 <!-- russt: changed these using drake's mesh_to_sdf -->
-                <pose>-0.00351257 0.00155128 0.0369668 0 0 0</pose>
-                <mass>0.8718110579379514</mass>
-                <inertia>
-                  <ixx>0.00398348</ixx>
-                  <ixy>2.33406e-05</ixy>
-                  <ixz>1.6376e-05</ixz>
-                  <iyy>0.000647219</iyy>
-                  <iyz>1.14248e-05</iyz>
-                  <izz>0.00411049</izz>
-                </inertia>
+                <origin xyz="-0.00351257 0.00155128 0.0369668"/>
+                <mass value="0.8718110579379514"/>
+                <inertia ixx="0.00398348"  ixy="2.33406e-05" ixz="1.6376e-05"
+                         iyy="0.000647219" iyz="1.14248e-05" izz="0.00411049"/>
                 <!-- these original values weren't physically valid
                 <mass value="1.4"/>
@@ -59,5 +53,5 @@
 					<mesh filename="package://QR/movo_description_drake/meshes/sensors/visual/kinect_one.obj" />
 				</geometry>
-        <material>
+        <material name="black">
           <color rgba="0.1788232 0.1788232 0.1788232 1"/>
         </material>
