Commit message: update gripper to hydroelastic

File: movo_common/movo_description/urdf/manipulation/jaco/jaco.urdf.xacro (robot description, xacro)
@@ -47,10 +47,10 @@
             <visual>
                 <geometry>
-                <mesh filename="package://QR/movo_description_drake/meshes/manipulation/jaco/visual/base.obj"/>
-                </geometry>
-            </visual>
-            <collision>
-                <geometry>
-                <mesh filename="package://QR/movo_description_drake/meshes/manipulation/jaco/collision/base.obj"/>
+                <mesh filename="package://movo_description/meshes/manipulation/jaco/visual/base.obj"/>
+                </geometry>
+            </visual>
+            <collision>
+                <geometry>
+                <mesh filename="package://movo_description/meshes/manipulation/jaco/collision/base.obj"/>
                 </geometry>
             </collision>
@@ -83,10 +83,10 @@
             <visual>
                 <geometry>
-                    <mesh filename="package://QR/movo_description_drake/meshes/manipulation/jaco/visual/shoulder.obj"/>
-                </geometry>
-            </visual>
-            <collision>
-                <geometry>
-                    <mesh filename="package://QR/movo_description_drake/meshes/manipulation/jaco/collision/shoulder.obj"/>
+                    <mesh filename="package://movo_description/meshes/manipulation/jaco/visual/shoulder.obj"/>
+                </geometry>
+            </visual>
+            <collision>
+                <geometry>
+                    <mesh filename="package://movo_description/meshes/manipulation/jaco/collision/shoulder.obj"/>
                 </geometry>
             </collision>
@@ -119,10 +119,10 @@
             <visual>
                 <geometry>
-                    <mesh filename="package://QR/movo_description_drake/meshes/manipulation/jaco/visual/upper_arm.obj"/>
-                </geometry>
-            </visual>
-            <collision>
-                <geometry>
-                    <mesh filename="package://QR/movo_description_drake/meshes/manipulation/jaco/collision/upper_arm.obj"/>
+                    <mesh filename="package://movo_description/meshes/manipulation/jaco/visual/upper_arm.obj"/>
+                </geometry>
+            </visual>
+            <collision>
+                <geometry>
+                    <mesh filename="package://movo_description/meshes/manipulation/jaco/collision/upper_arm.obj"/>
                 </geometry>
             </collision>
@@ -155,10 +155,10 @@
             <visual>
                 <geometry>
-                    <mesh filename="package://QR/movo_description_drake/meshes/manipulation/jaco/visual/forearm.obj"/>
-                </geometry>
-            </visual>
-            <collision>
-                <geometry>
-                    <mesh filename="package://QR/movo_description_drake/meshes/manipulation/jaco/collision/forearm.obj"/>
+                    <mesh filename="package://movo_description/meshes/manipulation/jaco/visual/forearm.obj"/>
+                </geometry>
+            </visual>
+            <collision>
+                <geometry>
+                    <mesh filename="package://movo_description/meshes/manipulation/jaco/collision/forearm.obj"/>
                 </geometry>
             </collision>
@@ -182,10 +182,10 @@
             <visual>
                 <geometry>
-                    <mesh filename="package://QR/movo_description_drake/meshes/manipulation/jaco/visual/wrist_1.obj"/>
-                </geometry>
-            </visual>
-            <collision>
-                <geometry>
-                    <mesh filename="package://QR/movo_description_drake/meshes/manipulation/jaco/collision/wrist_1.obj"/>
+                    <mesh filename="package://movo_description/meshes/manipulation/jaco/visual/wrist_1.obj"/>
+                </geometry>
+            </visual>
+            <collision>
+                <geometry>
+                    <mesh filename="package://movo_description/meshes/manipulation/jaco/collision/wrist_1.obj"/>
                 </geometry>
             </collision>
@@ -218,10 +218,10 @@
             <visual>
                 <geometry>
-                    <mesh filename="package://QR/movo_description_drake/meshes/manipulation/jaco/visual/wrist_2.obj"/>
-                </geometry>
-            </visual>
-            <collision>
-                <geometry>
-                    <mesh filename="package://QR/movo_description_drake/meshes/manipulation/jaco/collision/wrist_2.obj"/>
+                    <mesh filename="package://movo_description/meshes/manipulation/jaco/visual/wrist_2.obj"/>
+                </geometry>
+            </visual>
+            <collision>
+                <geometry>
+                    <mesh filename="package://movo_description/meshes/manipulation/jaco/collision/wrist_2.obj"/>
                 </geometry>
             </collision>
@@ -254,10 +254,10 @@
             <visual>
                 <geometry>
-                    <mesh filename="package://QR/movo_description_drake/meshes/manipulation/jaco/visual/kinova_actuator_gearing.obj"/>
-                </geometry>
-            </visual>
-            <collision>
-                <geometry>
-                    <mesh filename="package://QR/movo_description_drake/meshes/manipulation/jaco/collision/kinova_actuator_gearing.obj"/>
+                    <mesh filename="package://movo_description/meshes/manipulation/jaco/visual/kinova_actuator_gearing.obj"/>
+                </geometry>
+            </visual>
+            <collision>
+                <geometry>
+                    <mesh filename="package://movo_description/meshes/manipulation/jaco/collision/kinova_actuator_gearing.obj"/>
                 </geometry>
             </collision>

File: movo_common/movo_description/urdf/manipulation/jaco/jaco_7dof.urdf.xacro (robot description, xacro)
@@ -55,10 +55,10 @@
             <visual>
                 <geometry>
-                <mesh filename="package://QR/movo_description_drake/meshes/manipulation/jaco/visual/base.obj"/>
-                </geometry>
-            </visual>
-            <collision>
-                <geometry>
-                <mesh filename="package://QR/movo_description_drake/meshes/manipulation/jaco/collision/base.obj"/>
+                <mesh filename="package://movo_description/meshes/manipulation/jaco/visual/base.obj"/>
+                </geometry>
+            </visual>
+            <collision>
+                <geometry>
+                <mesh filename="package://movo_description/meshes/manipulation/jaco/collision/base.obj"/>
                 </geometry>
             </collision>
@@ -91,10 +91,10 @@
             <visual>
                 <geometry>
-                    <mesh filename="package://QR/movo_description_drake/meshes/manipulation/jaco/visual/shoulder_7dof.obj"/>
-                </geometry>
-            </visual>
-            <collision>
-                <geometry>
-                    <mesh filename="package://QR/movo_description_drake/meshes/manipulation/jaco/collision/shoulder_7dof.obj"/>
+                    <mesh filename="package://movo_description/meshes/manipulation/jaco/visual/shoulder_7dof.obj"/>
+                </geometry>
+            </visual>
+            <collision>
+                <geometry>
+                    <mesh filename="package://movo_description/meshes/manipulation/jaco/collision/shoulder_7dof.obj"/>
                 </geometry>
             </collision>
@@ -127,10 +127,10 @@
             <visual>
                 <geometry>
-                    <mesh filename="package://QR/movo_description_drake/meshes/manipulation/jaco/visual/arm_half_1.obj"/>
-                </geometry>
-            </visual>
-            <collision>
-                <geometry>
-                    <mesh filename="package://QR/movo_description_drake/meshes/manipulation/jaco/collision/arm_half_1.obj"/>
+                    <mesh filename="package://movo_description/meshes/manipulation/jaco/visual/arm_half_1.obj"/>
+                </geometry>
+            </visual>
+            <collision>
+                <geometry>
+                    <mesh filename="package://movo_description/meshes/manipulation/jaco/collision/arm_half_1.obj"/>
                 </geometry>
             </collision>
@@ -163,10 +163,10 @@
             <visual>
                 <geometry>
-                    <mesh filename="package://QR/movo_description_drake/meshes/manipulation/jaco/visual/arm_half_2.obj"/>
-                </geometry>
-            </visual>
-            <collision>
-                <geometry>
-                    <mesh filename="package://QR/movo_description_drake/meshes/manipulation/jaco/collision/arm_half_2.obj"/>
+                    <mesh filename="package://movo_description/meshes/manipulation/jaco/visual/arm_half_2.obj"/>
+                </geometry>
+            </visual>
+            <collision>
+                <geometry>
+                    <mesh filename="package://movo_description/meshes/manipulation/jaco/collision/arm_half_2.obj"/>
                 </geometry>
             </collision>
@@ -199,10 +199,10 @@
             <visual>
                 <geometry>
-                    <mesh filename="package://QR/movo_description_drake/meshes/manipulation/jaco/visual/forearm_7dof.obj"/>
-                </geometry>
-            </visual>
-            <collision>
-                <geometry>
-                    <mesh filename="package://QR/movo_description_drake/meshes/manipulation/jaco/collision/forearm_7dof.obj"/>
+                    <mesh filename="package://movo_description/meshes/manipulation/jaco/visual/forearm_7dof.obj"/>
+                </geometry>
+            </visual>
+            <collision>
+                <geometry>
+                    <mesh filename="package://movo_description/meshes/manipulation/jaco/collision/forearm_7dof.obj"/>
                 </geometry>
             </collision>
@@ -227,10 +227,10 @@
             <visual>
                 <geometry>
-                    <mesh filename="package://QR/movo_description_drake/meshes/manipulation/jaco/visual/wrist_spherical_1.obj"/>
-                </geometry>
-            </visual>
-            <collision>
-                <geometry>
-                    <mesh filename="package://QR/movo_description_drake/meshes/manipulation/jaco/collision/wrist_spherical_1.obj"/>
+                    <mesh filename="package://movo_description/meshes/manipulation/jaco/visual/wrist_spherical_1.obj"/>
+                </geometry>
+            </visual>
+            <collision>
+                <geometry>
+                    <mesh filename="package://movo_description/meshes/manipulation/jaco/collision/wrist_spherical_1.obj"/>
                 </geometry>
             </collision>
@@ -263,10 +263,10 @@
             <visual>
                 <geometry>
-                    <mesh filename="package://QR/movo_description_drake/meshes/manipulation/jaco/visual/wrist_spherical_2.obj"/>
-                </geometry>
-            </visual>
-            <collision>
-                <geometry>
-                    <mesh filename="package://QR/movo_description_drake/meshes/manipulation/jaco/collision/wrist_spherical_2.obj"/>
+                    <mesh filename="package://movo_description/meshes/manipulation/jaco/visual/wrist_spherical_2.obj"/>
+                </geometry>
+            </visual>
+            <collision>
+                <geometry>
+                    <mesh filename="package://movo_description/meshes/manipulation/jaco/collision/wrist_spherical_2.obj"/>
                 </geometry>
             </collision>
@@ -299,10 +299,10 @@
             <visual>
                 <geometry>
-                    <mesh filename="package://QR/movo_description_drake/meshes/manipulation/jaco/visual/kinova_actuator_gearing.obj"/>
-                </geometry>
-            </visual>
-            <collision>
-                <geometry>
-                    <mesh filename="package://QR/movo_description_drake/meshes/manipulation/jaco/collision/kinova_actuator_gearing.obj"/>
+                    <mesh filename="package://movo_description/meshes/manipulation/jaco/visual/kinova_actuator_gearing.obj"/>
+                </geometry>
+            </visual>
+            <collision>
+                <geometry>
+                    <mesh filename="package://movo_description/meshes/manipulation/jaco/collision/kinova_actuator_gearing.obj"/>
                 </geometry>
             </collision>

File: movo_common/movo_description/urdf/manipulation/kinova_grippers/kg2_gripper.urdf.xacro (robot description, xacro)
@@ -12,10 +12,10 @@
             <visual>
                 <geometry>
-                    <mesh filename="package://QR/movo_description_drake/meshes/manipulation/kinova_grippers/visual/kg2_base_link.dae"/>
-                </geometry>
-            </visual>
-            <collision>
-                <geometry>
-                    <mesh filename="package://QR/movo_description_drake/meshes/manipulation/kinova_grippers/collision/kg2_base_link.obj"/>
+                    <mesh filename="package://movo_description/meshes/manipulation/kinova_grippers/visual/kg2_base_link.dae"/>
+                </geometry>
+            </visual>
+            <collision>
+                <geometry>
+                    <mesh filename="package://movo_description/meshes/manipulation/kinova_grippers/collision/kg2_base_link.obj"/>
                 </geometry>
             </collision>
@@ -48,10 +48,10 @@
             <visual>
                 <geometry>
-                    <mesh filename="package://QR/movo_description_drake/meshes/manipulation/kinova_grippers/visual/finger_knuckle.dae"/>
-                </geometry>
-            </visual>
-            <collision>
-                <geometry>
-                    <mesh filename="package://QR/movo_description_drake/meshes/manipulation/kinova_grippers/collision/finger_knuckle.obj"/>
+                    <mesh filename="package://movo_description/meshes/manipulation/kinova_grippers/visual/finger_knuckle.dae"/>
+                </geometry>
+            </visual>
+            <collision>
+                <geometry>
+                    <mesh filename="package://movo_description/meshes/manipulation/kinova_grippers/collision/finger_knuckle.obj"/>
                 </geometry>
             </collision>
@@ -90,10 +90,10 @@
             <visual>
                 <geometry>
-                    <mesh filename="package://QR/movo_description_drake/meshes/manipulation/kinova_grippers/visual/finger_knuckle.dae"/>
-                </geometry>
-            </visual>
-            <collision>
-                <geometry>
-                    <mesh filename="package://QR/movo_description_drake/meshes/manipulation/kinova_grippers/collision/finger_knuckle.obj"/>
+                    <mesh filename="package://movo_description/meshes/manipulation/kinova_grippers/visual/finger_knuckle.dae"/>
+                </geometry>
+            </visual>
+            <collision>
+                <geometry>
+                    <mesh filename="package://movo_description/meshes/manipulation/kinova_grippers/collision/finger_knuckle.obj"/>
                 </geometry>
             </collision>
@@ -130,10 +130,10 @@
             <visual>
                 <geometry>
-                    <mesh filename="package://QR/movo_description_drake/meshes/manipulation/kinova_grippers/visual/finger_tip.dae"/>
-                </geometry>
-            </visual>
-            <collision>
-                <geometry>
-                    <mesh filename="package://QR/movo_description_drake/meshes/manipulation/kinova_grippers/collision/finger_tip.obj"/>
+                    <mesh filename="package://movo_description/meshes/manipulation/kinova_grippers/visual/finger_tip.dae"/>
+                </geometry>
+            </visual>
+            <collision>
+                <geometry>
+                    <mesh filename="package://movo_description/meshes/manipulation/kinova_grippers/collision/finger_tip.obj"/>
                 </geometry>
             </collision>
@@ -170,10 +170,10 @@
             <visual>
                 <geometry>
-                    <mesh filename="package://QR/movo_description_drake/meshes/manipulation/kinova_grippers/visual/finger_tip.dae"/>
-                </geometry>
-            </visual>
-            <collision>
-                <geometry>
-                    <mesh filename="package://QR/movo_description_drake/meshes/manipulation/kinova_grippers/collision/finger_tip.obj"/>
+                    <mesh filename="package://movo_description/meshes/manipulation/kinova_grippers/visual/finger_tip.dae"/>
+                </geometry>
+            </visual>
+            <collision>
+                <geometry>
+                    <mesh filename="package://movo_description/meshes/manipulation/kinova_grippers/collision/finger_tip.obj"/>
                 </geometry>
             </collision>
