Commit message: update gripper to hydroelastic

File: movo_common/movo_description/urdf/manipulation/kinova_grippers/kg3_gripper.urdf.xacro (robot description, xacro)
@@ -12,10 +12,10 @@
             <visual>
                 <geometry>
-                    <mesh filename="package://QR/movo_description_drake/meshes/manipulation/kinova_grippers/visual/kg3_base_link.dae"/>
-                </geometry>
-            </visual>
-            <collision>
-                <geometry>
-                    <mesh filename="package://QR/movo_description_drake/meshes/manipulation/kinova_grippers/collision/kg3_base_link.obj"/>
+                    <mesh filename="package://movo_description/meshes/manipulation/kinova_grippers/visual/kg3_base_link.dae"/>
+                </geometry>
+            </visual>
+            <collision>
+                <geometry>
+                    <mesh filename="package://movo_description/meshes/manipulation/kinova_grippers/collision/kg3_base_link.obj"/>
                 </geometry>
             </collision>
@@ -47,10 +47,10 @@
             <visual>
                 <geometry>
-                    <mesh filename="package://QR/movo_description_drake/meshes/manipulation/kinova_grippers/visual/finger_knuckle.dae"/>
-                </geometry>
-            </visual>
-            <collision>
-                <geometry>
-                    <mesh filename="package://QR/movo_description_drake/meshes/manipulation/kinova_grippers/collision/finger_knuckle.obj"/>
+                    <mesh filename="package://movo_description/meshes/manipulation/kinova_grippers/visual/finger_knuckle.dae"/>
+                </geometry>
+            </visual>
+            <collision>
+                <geometry>
+                    <mesh filename="package://movo_description/meshes/manipulation/kinova_grippers/collision/finger_knuckle.obj"/>
                 </geometry>
             </collision>
@@ -90,10 +90,10 @@
             <visual>
                 <geometry>
-                    <mesh filename="package://QR/movo_description_drake/meshes/manipulation/kinova_grippers/visual/finger_knuckle.dae"/>
-                </geometry>
-            </visual>
-            <collision>
-                <geometry>
-                    <mesh filename="package://QR/movo_description_drake/meshes/manipulation/kinova_grippers/collision/finger_knuckle.obj"/>
+                    <mesh filename="package://movo_description/meshes/manipulation/kinova_grippers/visual/finger_knuckle.dae"/>
+                </geometry>
+            </visual>
+            <collision>
+                <geometry>
+                    <mesh filename="package://movo_description/meshes/manipulation/kinova_grippers/collision/finger_knuckle.obj"/>
                 </geometry>
             </collision>
@@ -133,10 +133,10 @@
             <visual>
                 <geometry>
-                    <mesh filename="package://QR/movo_description_drake/meshes/manipulation/kinova_grippers/visual/finger_knuckle.dae"/>
-                </geometry>
-            </visual>
-            <collision>
-                <geometry>
-                    <mesh filename="package://QR/movo_description_drake/meshes/manipulation/kinova_grippers/collision/finger_knuckle.obj"/>
+                    <mesh filename="package://movo_description/meshes/manipulation/kinova_grippers/visual/finger_knuckle.dae"/>
+                </geometry>
+            </visual>
+            <collision>
+                <geometry>
+                    <mesh filename="package://movo_description/meshes/manipulation/kinova_grippers/collision/finger_knuckle.obj"/>
                 </geometry>
             </collision>
@@ -173,10 +173,10 @@
             <visual>
                 <geometry>
-                    <mesh filename="package://QR/movo_description_drake/meshes/manipulation/kinova_grippers/visual/finger_tip.dae"/>
-                </geometry>
-            </visual>
-            <collision>
-                <geometry>
-                    <mesh filename="package://QR/movo_description_drake/meshes/manipulation/kinova_grippers/collision/finger_tip.obj"/>
+                    <mesh filename="package://movo_description/meshes/manipulation/kinova_grippers/visual/finger_tip.dae"/>
+                </geometry>
+            </visual>
+            <collision>
+                <geometry>
+                    <mesh filename="package://movo_description/meshes/manipulation/kinova_grippers/collision/finger_tip.obj"/>
                 </geometry>
             </collision>
@@ -213,10 +213,10 @@
             <visual>
                 <geometry>
-                    <mesh filename="package://QR/movo_description_drake/meshes/manipulation/kinova_grippers/visual/finger_tip.dae"/>
-                </geometry>
-            </visual>
-            <collision>
-                <geometry>
-                    <mesh filename="package://QR/movo_description_drake/meshes/manipulation/kinova_grippers/collision/finger_tip.obj"/>
+                    <mesh filename="package://movo_description/meshes/manipulation/kinova_grippers/visual/finger_tip.dae"/>
+                </geometry>
+            </visual>
+            <collision>
+                <geometry>
+                    <mesh filename="package://movo_description/meshes/manipulation/kinova_grippers/collision/finger_tip.obj"/>
                 </geometry>
             </collision>
@@ -253,10 +253,10 @@
             <visual>
                 <geometry>
-                    <mesh filename="package://QR/movo_description_drake/meshes/manipulation/kinova_grippers/visual/finger_tip.dae"/>
-                </geometry>
-            </visual>
-            <collision>
-                <geometry>
-                    <mesh filename="package://QR/movo_description_drake/meshes/manipulation/kinova_grippers/collision/finger_tip.obj"/>
+                    <mesh filename="package://movo_description/meshes/manipulation/kinova_grippers/visual/finger_tip.dae"/>
+                </geometry>
+            </visual>
+            <collision>
+                <geometry>
+                    <mesh filename="package://movo_description/meshes/manipulation/kinova_grippers/collision/finger_tip.obj"/>
                 </geometry>
             </collision>

File: movo_common/movo_description/urdf/manipulation/robotiq/robotiq_85_gripper.urdf (robot description, URDF)
Before this commit: robot robotiq85_gripper, 10 links, 9 joints
Links:
- link gripper_finger1_finger_tip_link: geometry collision box size=0.0375 0.00675 0.022; visual mesh filename=package://movo_description/meshes/manipulation/robotiq/visu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

File: movo_common/movo_description/urdf/movo_components/movo_base.urdf.xacro (robot description, xacro)
@@ -104,5 +104,5 @@
             <collision>
 				<geometry>
-					<mesh filename="package://QR/movo_description_drake/meshes/movo_components/collision/vector_base_collision.obj" />
+					<mesh filename="package://movo_description/meshes/movo_components/collision/vector_base_collision.obj" />
 				</geometry>
 			</collision>
@@ -111,5 +111,5 @@
 				<origin xyz="0 0 0" rpy="0 0 0" />
 				<geometry>
-					<mesh filename="package://QR/movo_description_drake/meshes/movo_components/visual/vector_base.obj" />
+					<mesh filename="package://movo_description/meshes/movo_components/visual/vector_base.obj" />
 				</geometry>
         <material name="black">
@@ -140,5 +140,5 @@
             <collision>
 				<geometry>
-					<mesh filename="package://QR/movo_description_drake/meshes/movo_components/collision/movo_fixed_body_collision.obj" />
+					<mesh filename="package://movo_description/meshes/movo_components/collision/movo_fixed_body_collision.obj" />
 				</geometry>
 			</collision>
@@ -146,5 +146,5 @@
 				<origin xyz="0 0 0" rpy="0 0 0" />
 				<geometry>
-					<mesh filename="package://QR/movo_description_drake/meshes/movo_components/collision/movo_fixed_body_collision.obj" />
+					<mesh filename="package://movo_description/meshes/movo_components/collision/movo_fixed_body_collision.obj" />
 				</geometry>
 			</visual>
@@ -166,5 +166,5 @@
 		    <visual>
 			    <geometry>
-				    <mesh filename="package://QR/movo_description_drake/meshes/movo_components/collision/movo_upper_body_collision.obj" />
+				    <mesh filename="package://movo_description/meshes/movo_components/collision/movo_upper_body_collision.obj" />
 			    </geometry>
 		    </visual>-->
@@ -172,5 +172,5 @@
 		    <collision>
 			    <geometry>
-				    <mesh filename="package://QR/movo_description_drake/meshes/movo_components/collision/movo_upper_body_collision.obj" />
+				    <mesh filename="package://movo_description/meshes/movo_components/collision/movo_upper_body_collision.obj" />
 			    </geometry>
 		    </collision>

File: movo_common/movo_description/urdf/movo_components/movo_body.urdf.xacro (robot description, xacro)
@@ -54,5 +54,5 @@
 				<origin xyz="0 0 0" rpy="0 0 0" />
 				<geometry>
-					<mesh filename="package://QR/movo_description_drake/meshes/movo_body/movo_lower_body.obj" />
+					<mesh filename="package://movo_description/meshes/movo_body/movo_lower_body.obj" />
 				</geometry>
         <material name="black">
@@ -84,5 +84,5 @@
 				<origin xyz="0 0 0" rpy="0 0 0" />
 				<geometry>
-					<mesh filename="package://QR/movo_description_drake/meshes/movo_body/movo_upper_body.obj" />
+					<mesh filename="package://movo_description/meshes/movo_body/movo_upper_body.obj" />
 				</geometry>
         <material name="black">
@@ -123,5 +123,5 @@
 				<origin xyz="0 0 0" rpy="0 0 0" />
 				<geometry>
-					<mesh filename="package://QR/movo_description_drake/meshes/movo_body/movo_mid_body.obj" />
+					<mesh filename="package://movo_description/meshes/movo_body/movo_mid_body.obj" />
 				</geometry>
         <material name="black">

File: movo_common/movo_description/urdf/movo_components/movo_pan_tilt.urdf.xacro (robot description, xacro)
@@ -39,5 +39,5 @@
 			<visual>
 				<geometry>
-					<mesh filename="package://QR/movo_description_drake/meshes/pan_tilt/visual/pan_tilt_base.obj" />
+					<mesh filename="package://movo_description/meshes/pan_tilt/visual/pan_tilt_base.obj" />
 				</geometry>
         <material name="black">
@@ -47,5 +47,5 @@
 			<collision>
 				<geometry>
-					<mesh filename="package://QR/movo_description_drake/meshes/pan_tilt/collision/pan_tilt_base.obj" />
+					<mesh filename="package://movo_description/meshes/pan_tilt/collision/pan_tilt_base.obj" />
 				</geometry>
 			</collision>
@@ -77,5 +77,5 @@
 			<visual>
 				<geometry>
-					<mesh filename="package://QR/movo_description_drake/meshes/pan_tilt/visual/pan_link.obj" />
+					<mesh filename="package://movo_description/meshes/pan_tilt/visual/pan_link.obj" />
 				</geometry>
         <material name="black">
@@ -86,5 +86,5 @@
 			    <origin xyz="0 0 0" rpy="0 0 0" />
 				<geometry>
-					<mesh filename="package://QR/movo_description_drake/meshes/pan_tilt/collision/pan_link.obj" />
+					<mesh filename="package://movo_description/meshes/pan_tilt/collision/pan_link.obj" />
 				</geometry>
 			</collision>
@@ -116,5 +116,5 @@
 			<visual>
 				<geometry>
-					<mesh filename="package://QR/movo_description_drake/meshes/pan_tilt/visual/tilt_link.obj" />
+					<mesh filename="package://movo_description/meshes/pan_tilt/visual/tilt_link.obj" />
 				</geometry>
         <material name="black">
@@ -124,5 +124,5 @@
 			<collision>
 				<geometry>
-					<mesh filename="package://QR/movo_description_drake/meshes/pan_tilt/collision/tilt_link.obj" />
+					<mesh filename="package://movo_description/meshes/pan_tilt/collision/tilt_link.obj" />
 				</geometry>
 			</collision>

File: movo_common/movo_description/urdf/movo_components/proto2_arm_mount.urdf.xacro (robot description, xacro)
@@ -37,10 +37,10 @@
 			<visual>
 				<geometry>
-					<mesh filename="package://QR/movo_description_drake/meshes/proto2/visual/proto2_arm_mount.dae" />
+					<mesh filename="package://movo_description/meshes/proto2/visual/proto2_arm_mount.dae" />
 				</geometry>
 			</visual>
 			<collision>
 				<geometry>
-					<mesh filename="package://QR/movo_description_drake/meshes/proto2/collision/proto2_arm_mount_collision.dae" />
+					<mesh filename="package://movo_description/meshes/proto2/collision/proto2_arm_mount_collision.dae" />
 				</geometry>
 			</collision>

File: movo_common/movo_description/urdf/movo_components/proto2_base.urdf.xacro (robot description, xacro)
@@ -51,5 +51,5 @@
             <collision>
 				<geometry>
-					<mesh filename="package://QR/movo_description_drake/meshes/proto2/collision/proto2_base_collision.dae" />
+					<mesh filename="package://movo_description/meshes/proto2/collision/proto2_base_collision.dae" />
 				</geometry>
 			</collision>
@@ -57,5 +57,5 @@
 				<origin xyz="0 0 0" rpy="0 0 0" />
 				<geometry>
-					<mesh filename="package://QR/movo_description_drake/meshes/proto2/visual/proto2_base.dae"  />
+					<mesh filename="package://movo_description/meshes/proto2/visual/proto2_base.dae"  />
 				</geometry>
 			</visual>

File: movo_common/movo_description/urdf/movo_components/proto2_frame.urdf.xacro (robot description, xacro)
@@ -37,10 +37,10 @@
 			<visual>
 				<geometry>
-					<mesh filename="package://QR/movo_description_drake/meshes/proto2/visual/proto2_frame.dae" />
+					<mesh filename="package://movo_description/meshes/proto2/visual/proto2_frame.dae" />
 				</geometry>
 			</visual>
 			<collision>
 				<geometry>
-					<mesh filename="package://QR/movo_description_drake/meshes/proto2/collision/proto2_frame_collision.dae" />
+					<mesh filename="package://movo_description/meshes/proto2/collision/proto2_frame_collision.dae" />
 				</geometry>
 			</collision>

File: movo_common/movo_description/urdf/sensors/kinect_one_sensor.urdf.xacro (robot description, xacro)
@@ -51,5 +51,5 @@
 			<visual>
 				<geometry>
-					<mesh filename="package://QR/movo_description_drake/meshes/sensors/visual/kinect_one.obj" />
+					<mesh filename="package://movo_description/meshes/sensors/visual/kinect_one.obj" />
 				</geometry>
         <material name="black">
@@ -59,5 +59,5 @@
 			<collision>
 				<geometry>
-					<mesh filename="package://QR/movo_description_drake/meshes/sensors/collision/kinect_one_collision.obj" />
+					<mesh filename="package://movo_description/meshes/sensors/collision/kinect_one_collision.obj" />
 				</geometry>
 			</collision>

File: movo_common/movo_description/urdf/sensors/sick_tim.urdf.xacro (robot description, xacro)
@@ -37,5 +37,5 @@
 <!--            <visual>
                 <geometry>
-                    <mesh filename="package://QR/movo_description_drake/meshes/sensors/visual/sick_tim.obj" />
+                    <mesh filename="package://movo_description/meshes/sensors/visual/sick_tim.obj" />
                 </geometry>
             </visual> -->
@@ -46,4 +46,16 @@
             </collision>
         </link>
+        <joint name="${laser_prefix}_laser_joint_virtual" type="fixed">
+          <origin rpy="-1.570795 0 -1.570795" xyz="0.0 0 0"/>
+          <parent link="${laser_prefix}_laser_link"/>
+          <child link="${laser_prefix}_laser_link_virtual"/>
+        </joint>
+        <link name="${laser_prefix}_laser_link_virtual">
+          <collision>
+            <geometry>
+              <box size="0.001 0.001 0.001"/>
+            </geometry>
+          </collision>
+          </link>
         <gazebo reference="${laser_prefix}_laser_link">
             <sensor type="ray" name="${laser_prefix}_laser">
